File: kicad/sramBoard/1BIT_CELL.kicad_sch (KiCad schematic)
At the start: 8 parts, among them Q1 NMOS, Q2 NMOS, Q3 PMOS, Q4 NMOS, Q5 PMOS, Q6 NMOS, Q7 NMOS, Q8 NMOS

Commit message: Initial ram board schematic
Parts:
- Q1, Q2, Q4, Q6, Q7, Q8: footprint Package_DFN_QFN:Nordic_AQFN-94-1EP_7x7mm_P0.4mm -> Package_TO_SOT_SMD:SOT-23
- Q3, Q5: footprint (none) -> Package_TO_SOT_SMD:SOT-23
Changed lines of the file:
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@@
 			)
 		)
-		(property "Footprint" ""
+		(property "Footprint" "Package_TO_SOT_SMD:SOT-23"
 			(at 123.19 82.55 0)
 			(hide yes)
@@
 			)
 		)
-		(property "Footprint" "Package_DFN_QFN:Nordic_AQFN-94-1EP_7x7mm_P0.4mm"
+		(property "Footprint" "Package_TO_SOT_SMD:SOT-23"
 			(at 77.47 92.71 0)
 			(hide yes)
@@
 			)
 		)
-		(property "Footprint" "Package_DFN_QFN:Nordic_AQFN-94-1EP_7x7mm_P0.4mm"
+		(property "Footprint" "Package_TO_SOT_SMD:SOT-23"
 			(at 107.95 95.25 0)
 			(hide yes)
@@
 			)
 		)
-		(property "Footprint" "Package_DFN_QFN:Nordic_AQFN-94-1EP_7x7mm_P0.4mm"
+		(property "Footprint" "Package_TO_SOT_SMD:SOT-23"
 			(at 123.19 95.25 0)
 			(hide yes)
@@
 			)
 		)
-		(property "Footprint" "Package_DFN_QFN:Nordic_AQFN-94-1EP_7x7mm_P0.4mm"
+		(property "Footprint" "Package_TO_SOT_SMD:SOT-23"
 			(at 152.4 90.17 0)
 			(hide yes)
@@
 			)
 		)
-		(property "Footprint" "Package_DFN_QFN:Nordic_AQFN-94-1EP_7x7mm_P0.4mm"
+		(property "Footprint" "Package_TO_SOT_SMD:SOT-23"
 			(at 72.39 92.71 0)
 			(hide yes)
@@
 			)
 		)
-		(property "Footprint" ""
+		(property "Footprint" "Package_TO_SOT_SMD:SOT-23"
 			(at 107.95 82.55 0)
 			(hide yes)
@@
 			)
 		)
-		(property "Footprint" "Package_DFN_QFN:Nordic_AQFN-94-1EP_7x7mm_P0.4mm"
+		(property "Footprint" "Package_TO_SOT_SMD:SOT-23"
 			(at 157.48 90.17 0)
 			(hide yes)
