File: kicad/sramBoard/sramBoard.kicad_pcb (KiCad board)
At the start: 4 copper layers, 180 x 180 mm, 1225 parts, among them J1 Conn_02x20_Top_Bottom, Q1 NMOS, Q10 NMOS, Q100 NMOS, Q1000 NMOS, Q1001 NMOS, Q1002 NMOS, Q1003 PMOS, Q1004 NMOS, Q1005 PMOS, Q1006 NMOS, Q1007 NMOS, Q1008 NMOS, Q1009 NMOS, Q101 PMOS, Q1010 NMOS, Q1011 PMOS, Q1012 NMOS, Q1013 PMOS, Q1014 NMOS, Q1015 NMOS, Q1016 NMOS, Q1017 NMOS, Q1018 NMOS, Q1019 PMOS, Q102 NMOS, Q1020 NMOS, Q1021 PMOS, Q1022 NMOS, Q1023 NMOS, Q1024 NMOS, Q1025 PMOS, Q1026 NMOS, Q1027 PMOS, Q1028 NMOS, Q1029 PMOS, Q103 NMOS, Q1030 NMOS, Q1031 PMOS, Q1032 NMOS, Q1033 PMOS, Q1034 PMOS, Q1035 PMOS, Q1036 PMOS, Q1037 PMOS, Q1038 NMOS, Q1039 NMOS, Q104 NMOS, Q1040 NMOS, Q1041 NMOS, Q1042 NMOS, Q1043 PMOS, Q1044 PMOS, Q1045 PMOS, Q1046 PMOS, Q1047 PMOS, Q1048 NMOS, Q1049 NMOS, Q105 NMOS, Q1050 NMOS, Q1051 NMOS, Q1052 NMOS, Q1053 PMOS, Q1054 PMOS, Q1055 PMOS, Q1056 PMOS, Q1057 PMOS, Q1058 NMOS, Q1059 NMOS, Q106 NMOS, Q1060 NMOS, Q1061 NMOS, Q1062 NMOS, Q1063 PMOS, Q1064 PMOS, Q1065 PMOS, Q1066 PMOS, Q1067 PMOS, Q1068 NMOS, Q1069 NMOS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

Commit message: did more simulation work
Routing:
- net /8BIT_ROW/BL_{7}: track 352.9 -> 247.4 mm
- net /8BIT_ROW/BL_{2}: track 371.5 -> 269.5 mm
- net /8BIT_ROW/~{BL_{7}}: track 369.5 -> 270.3 mm
- net /8BIT_ROW/~{BL_{6}}: track 339.2 -> 240.6 mm
- net /8BIT_ROW/~{BL_{3}}: track 361.1 -> 262.8 mm
- net /8BIT_ROW/~{BL_{2}}: track 370.6 -> 272.4 mm
- net /8BIT_ROW/BL_{3}: track 364.9 -> 266.7 mm
- net /8BIT_ROW/BL_{6}: track 332.0 -> 238.4 mm
- net /8BIT_ROW/~{BL_{5}}: track 330.8 -> 237.3 mm
- net /8BIT_ROW/BL_{5}: track 336.3 -> 243.0 mm
- net /8BIT_ROW/~{BL_{4}}: track 340.0 -> 246.9 mm
- net /8BIT_ROW/BL_{4}: track 345.0 -> 252.0 mm
