File: kicad/sramBoard/sramBoard.kicad_pcb (KiCad board)
At the start: 4 copper layers, 155 x 170 mm, 2013 parts, among them J1 Conn_02x20_Top_Bottom, J10 Conn_01x02_Pin, J100 Conn_01x02_Pin, J101 Conn_01x02_Pin, J102 Conn_01x02_Pin, J103 Conn_01x02_Pin, J104 Conn_01x02_Pin, J105 Conn_01x02_Pin, J106 Conn_01x02_Pin, J107 Conn_01x02_Pin, J108 Conn_01x02_Pin, J109 Conn_01x02_Pin, J11 Conn_01x02_Pin, J110 Conn_01x02_Pin, J111 Conn_01x02_Pin, J112 Conn_01x02_Pin, J113 Conn_01x02_Pin, J114 Conn_01x02_Pin, J115 Conn_01x02_Pin, J116 Conn_01x02_Pin, J117 Conn_01x02_Pin, J118 Conn_01x02_Pin, J119 Conn_01x02_Pin, J12 Conn_01x02_Pin, J120 Conn_01x02_Pin, J121 Conn_01x02_Pin, J122 Conn_01x02_Pin, J123 Conn_01x02_Pin, J124 Conn_01x02_Pin, J125 Conn_01x02_Pin, J126 Conn_01x02_Pin, J127 Conn_01x02_Pin, J128 Conn_01x02_Pin, J129 Conn_01x02_Pin, J13 Conn_01x02_Pin, J14 Conn_01x02_Pin, J15 Conn_01x02_Pin, J16 Conn_01x02_Pin, J17 Conn_01x02_Pin, J18 Conn_01x02_Pin, J19 Conn_01x02_Pin, J2 Conn_01x02_Pin, J20 Conn_01x02_Pin, J21 Conn_01x02_Pin, J22 Conn_01x02_Pin, J23 Conn_01x02_Pin, J24 Conn_01x02_Pin, J25 Conn_01x02_Pin, J26 Conn_01x02_Pin, J27 Conn_01x02_Pin, J28 Conn_01x02_Pin, J29 Conn_01x02_Pin, J3 Conn_01x02_Pin, J30 Conn_01x02_Pin, J31 Conn_01x02_Pin, J32 Conn_01x02_Pin, J33 Conn_01x02_Pin, J34 Conn_01x02_Pin, J35 Conn_01x02_Pin, J36 Conn_01x02_Pin, J37 Conn_01x02_Pin, J38 Conn_01x02_Pin, J39 Conn_01x02_Pin, J4 Conn_01x02_Pin, J40 Conn_01x02_Pin, J41 Conn_01x02_Pin, J42 Conn_01x02_Pin, J43 Conn_01x02_Pin, J44 Conn_01x02_Pin, J45 Conn_01x02_Pin, J46 Conn_01x02_Pin, J47 Conn_01x02_Pin, J48 Conn_01x02_Pin, J49 Conn_01x02_Pin, J5 Conn_01x02_Pin, J50 Conn_01x02_Pin, J51 Conn_01x02_Pin, J52 Conn_01x02_Pin, J53 Conn_01x02_Pin, J54 Conn_01x02_Pin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

Commit message: update bom, add more capacitors
Parts:
- added J130: Conn_01x01_Pin, Connector_Wire:Wire_Pad_18AWG_stranded, F.Cu at (207.8, 193.6)
- added J131: Conn_01x01_Pin, Connector_Wire:Wire_Pad_18AWG_stranded, F.Cu at (218.6, 176.7)
- added J132: Conn_01x01_Pin, Connector_Wire:Wire_Pad_18AWG_stranded, F.Cu at (218.6, 166.7)
- added J133: Conn_01x01_Pin, Connector_Wire:Wire_Pad_18AWG_stranded, F.Cu at (218.6, 156.7)
- added J134: Conn_01x01_Pin, Connector_Wire:Wire_Pad_18AWG_stranded, F.Cu at (218.2, 118.0)
- added J135: Conn_01x01_Pin, Connector_Wire:Wire_Pad_18AWG_stranded, F.Cu at (218.1, 126.5)
- added J136: Conn_01x01_Pin, Connector_Wire:Wire_Pad_18AWG_stranded, F.Cu at (218.1, 136.5)
- added J137: Conn_01x01_Pin, Connector_Wire:Wire_Pad_18AWG_stranded, F.Cu at (218.6, 146.2)
- R101, R103, R105, R107, R109, R11, R111, R113, R115, R117, R119, R121, R123, R125, R127, R129, R13, R131, R133, R135, R137, R139, R141, R143, R145, R147, R149, R15, R151, R153, R155, R157, R159, R161, R163, R165, R167, R169, R17, R171, R173, R175, R177, R179, R181, R183, R185, R187, R189, R19, R191, R193, R195, R197, R199, R201, R203, R205, R207, R209, R21, R211, R213, R215, R217, R219, R221, R223, R225, R227, R229, R23, R231, R233, R235, R237, R239, R241, R243, R245, R247, R249, R25, R251, R253, R255, R257, R259, R261, R27, R29, R31, R33, R35, R37, R39, R41, R43, R45, R47, R49, R51, R53, R55, R57, R59, R61, R63, R65, R67, R69, R7, R71, R73, R75, R77, R79, R81, R83, R85, R87, R89, R9, R91, R93, R95, R97, R99: value 360R -> 180R
- moved R3 0.89 mm to (216.4, 182.3)
Routing:
- net /8BIT_ROW/~{BL_{1}}: track 301.8 -> 302.6 mm
- net GND: vias 420 -> 421
- net +5V: vias 214 -> 215
