File: kicad/sramBoard/1_16_5V_DEMUX_NOTOUT/1_16_5V_DEMUX_NOTOUT.kicad_sch (KiCad schematic)
At the start: 0 parts

Commit message: first pcb deign for main boards
Other:
- sheet 5VNOT: file 1_16_5V_DEMUX_NOTOUT/5VNOT/5VNOT.kicad_sch -> 5VNOT/5VNOT.kicad_sch
- sheet 5VNOT1: file 1_16_5V_DEMUX_NOTOUT/5VNOT/5VNOT.kicad_sch -> 5VNOT/5VNOT.kicad_sch
- sheet 5VNOT2: file 1_16_5V_DEMUX_NOTOUT/5VNOT/5VNOT.kicad_sch -> 5VNOT/5VNOT.kicad_sch
- sheet 5VNOT3: file 1_16_5V_DEMUX_NOTOUT/5VNOT/5VNOT.kicad_sch -> 5VNOT/5VNOT.kicad_sch
- sheet 5V_5NAND: file 1_16_5V_DEMUX_NOTOUT/5V_NAND/5V_5NAND.kicad_sch -> 5V_5NAND/5V_5NAND.kicad_sch
- sheet 5V_5NAND1: file 1_16_5V_DEMUX_NOTOUT/5V_NAND/5V_5NAND.kicad_sch -> 5V_5NAND/5V_5NAND.kicad_sch
- sheet 5V_5NAND10: file 1_16_5V_DEMUX_NOTOUT/5V_NAND/5V_5NAND.kicad_sch -> 5V_5NAND/5V_5NAND.kicad_sch
- sheet 5V_5NAND11: file 1_16_5V_DEMUX_NOTOUT/5V_NAND/5V_5NAND.kicad_sch -> 5V_5NAND/5V_5NAND.kicad_sch
- sheet 5V_5NAND12: file 1_16_5V_DEMUX_NOTOUT/5V_NAND/5V_5NAND.kicad_sch -> 5V_5NAND/5V_5NAND.kicad_sch
- sheet 5V_5NAND13: file 1_16_5V_DEMUX_NOTOUT/5V_NAND/5V_5NAND.kicad_sch -> 5V_5NAND/5V_5NAND.kicad_sch
- sheet 5V_5NAND14: file 1_16_5V_DEMUX_NOTOUT/5V_NAND/5V_5NAND.kicad_sch -> 5V_5NAND/5V_5NAND.kicad_sch
- sheet 5V_5NAND15: file 1_16_5V_DEMUX_NOTOUT/5V_NAND/5V_5NAND.kicad_sch -> 5V_5NAND/5V_5NAND.kicad_sch
- sheet 5V_5NAND2: file 1_16_5V_DEMUX_NOTOUT/5V_NAND/5V_5NAND.kicad_sch -> 5V_5NAND/5V_5NAND.kicad_sch
- sheet 5V_5NAND3: file 1_16_5V_DEMUX_NOTOUT/5V_NAND/5V_5NAND.kicad_sch -> 5V_5NAND/5V_5NAND.kicad_sch
- sheet 5V_5NAND4: file 1_16_5V_DEMUX_NOTOUT/5V_NAND/5V_5NAND.kicad_sch -> 5V_5NAND/5V_5NAND.kicad_sch
- sheet 5V_5NAND5: file 1_16_5V_DEMUX_NOTOUT/5V_NAND/5V_5NAND.kicad_sch -> 5V_5NAND/5V_5NAND.kicad_sch
- sheet 5V_5NAND6: file 1_16_5V_DEMUX_NOTOUT/5V_NAND/5V_5NAND.kicad_sch -> 5V_5NAND/5V_5NAND.kicad_sch
- sheet 5V_5NAND7: file 1_16_5V_DEMUX_NOTOUT/5V_NAND/5V_5NAND.kicad_sch -> 5V_5NAND/5V_5NAND.kicad_sch
- sheet 5V_5NAND8: file 1_16_5V_DEMUX_NOTOUT/5V_NAND/5V_5NAND.kicad_sch -> 5V_5NAND/5V_5NAND.kicad_sch
- sheet 5V_5NAND9: file 1_16_5V_DEMUX_NOTOUT/5V_NAND/5V_5NAND.kicad_sch -> 5V_5NAND/5V_5NAND.kicad_sch
Changed lines of the file:
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@@
 			)
 		)
-		(property "Sheetfile" "1_16_5V_DEMUX_NOTOUT/5V_NAND/5V_5NAND.kicad_sch"
+		(property "Sheetfile" "5V_5NAND/5V_5NAND.kicad_sch"
 			(at 206.3246 95.25 90)
 			(show_name no)
@@
 				(path "/13380198-0e23-4241-a844-cca11526fb8d/a0132d23-2efe-4baa-845a-d59f49944fa0"
 					(page "160")
+				)
+			)
+			(project "1_16_5V_DEMUX_NOTOUT"
+				(path "/64c295c1-a690-461e-ae3b-f66cfdb6e72a"
+					(page "18")
 				)
 			)
@@
 			)
 		)
-		(property "Sheetfile" "1_16_5V_DEMUX_NOTOUT/5VNOT/5VNOT.kicad_sch"
+		(property "Sheetfile" "5VNOT/5VNOT.kicad_sch"
 			(at 53.34 65.3546 0)
 			(show_name no)
@@
 				(path "/13380198-0e23-4241-a844-cca11526fb8d/a0132d23-2efe-4baa-845a-d59f49944fa0"
 					(page "150")
+				)
+			)
+			(project "1_16_5V_DEMUX_NOTOUT"
+				(path "/64c295c1-a690-461e-ae3b-f66cfdb6e72a"
+					(page "2")
 				)
 			)
@@
 			)
 		)
-		(property "Sheetfile" "1_16_5V_DEMUX_NOTOUT/5V_NAND/5V_5NAND.kicad_sch"
+		(property "Sheetfile" "5V_5NAND/5V_5NAND.kicad_sch"
 			(at 135.2046 95.25 90)
 			(show_name no)
@@
 				(path "/13380198-0e23-4241-a844-cca11526fb8d/a0132d23-2efe-4baa-845a-d59f49944fa0"
 					(page "162")
+				)
+			)
+			(project "1_16_5V_DEMUX_NOTOUT"
+				(path "/64c295c1-a690-461e-ae3b-f66cfdb6e72a"
+					(page "10")
 				)
 			)
@@
 			)
 		)
-		(property "Sheetfile" "1_16_5V_DEMUX_NOTOUT/5V_NAND/5V_5NAND.kicad_sch"
+		(property "Sheetfile" "5V_5NAND/5V_5NAND.kicad_sch"
 			(at 136.4746 45.72 90)
 			(show_name no)
@@
 				(path "/13380198-0e23-4241-a844-cca11526fb8d/a0132d23-2efe-4baa-845a-d59f49944fa0"
 					(page "155")
+				)
+			)
+			(project "1_16_5V_DEMUX_NOTOUT"
+				(path "/64c295c1-a690-461e-ae3b-f66cfdb6e72a"
+					(page "11")
 				)
 			)
@@
 			)
 		)
-		(property "Sheetfile" "1_16_5V_DEMUX_NOTOUT/5V_NAND/5V_5NAND.kicad_sch"
+		(property "Sheetfile" "5V_5NAND/5V_5NAND.kicad_sch"
 			(at 224.1046 95.25 90)
 			(show_name no)
@@
 				(path "/13380198-0e23-4241-a844-cca11526fb8d/a0132d23-2efe-4baa-845a-d59f49944fa0"
 					(page "159")
+				)
+			)
+			(project "1_16_5V_DEMUX_NOTOUT"
+				(path "/64c295c1-a690-461e-ae3b-f66cfdb6e72a"
+					(page "20")
 				)
 			)
@@
 			)
 		)
-		(property "Sheetfile" "1_16_5V_DEMUX_NOTOUT/5V_NAND/5V_5NAND.kicad_sch"
+		(property "Sheetfile" "5V_5NAND/5V_5NAND.kicad_sch"
 			(at 99.6446 95.25 90)
 			(show_name no)
@@
 				(path "/13380198-0e23-4241-a844-cca11526fb8d/a0132d23-2efe-4baa-845a-d59f49944fa0"
 					(page "152")
+				)
+			)
+			(project "1_16_5V_DEMUX_NOTOUT"
+				(path "/64c295c1-a690-461e-ae3b-f66cfdb6e72a"
+					(page "6")
 				)
 			)
@@
 			)
 		)
-		(property "Sheetfile" "1_16_5V_DEMUX_NOTOUT/5VNOT/5VNOT.kicad_sch"
+		(property "Sheetfile" "5VNOT/5VNOT.kicad_sch"
 			(at 53.34 72.9746 0)
 			(show_name no)
@@
 				(path "/13380198-0e23-4241-a844-cca11526fb8d/a0132d23-2efe-4baa-845a-d59f49944fa0"
 					(page "149")
+				)
+			)
+			(project "1_16_5V_DEMUX_NOTOUT"
+				(path "/64c295c1-a690-461e-ae3b-f66cfdb6e72a"
+					(page "3")
 				)
 			)
@@
 			)
 		)
-		(property "Sheetfile" "1_16_5V_DEMUX_NOTOUT/5VNOT/5VNOT.kicad_sch"
+		(property "Sheetfile" "5VNOT/5VNOT.kicad_sch"
 			(at 53.34 80.5946 0)
 			(show_name no)
@@
 				(path "/13380198-0e23-4241-a844-cca11526fb8d/a0132d23-2efe-4baa-845a-d59f49944fa0"
 					(page "147")
+				)
+			)
+			(project "1_16_5V_DEMUX_NOTOUT"
+				(path "/64c295c1-a690-461e-ae3b-f66cfdb6e72a"
+					(page "4")
 				)
 			)
@@
 			)
 		)
-		(property "Sheetfile" "1_16_5V_DEMUX_NOTOUT/5V_NAND/5V_5NAND.kicad_sch"
+		(property "Sheetfile" "5V_5NAND/5V_5NAND.kicad_sch"
 			(at 207.5946 45.72 90)
 			(show_name no)
@@
 				(path "/13380198-0e23-4241-a844-cca11526fb8d/a0132d23-2efe-4baa-845a-d59f49944fa0"
 					(page "166")
+				)
+			)
+			(project "1_16_5V_DEMUX_NOTOUT"
+				(path "/64c295c1-a690-461e-ae3b-f66cfdb6e72a"
+					(page "19")
 				)
 			)
@@
 			)
 		)
-		(property "Sheetfile" "1_16_5V_DEMUX_NOTOUT/5V_NAND/5V_5NAND.kicad_sch"
+		(property "Sheetfile" "5V_5NAND/5V_5NAND.kicad_sch"
 			(at 154.2546 45.72 90)
 			(show_name no)
@@
 				(path "/13380198-0e23-4241-a844-cca11526fb8d/a0132d23-2efe-4baa-845a-d59f49944fa0"
 					(page "156")
+				)
+			)
+			(project "1_16_5V_DEMUX_NOTOUT"
+				(path "/64c295c1-a690-461e-ae3b-f66cfdb6e72a"
+					(page "13")
 				)
 			)
@@
 			)
 		)
-		(property "Sheetfile" "1_16_5V_DEMUX_NOTOUT/5V_NAND/5V_5NAND.kicad_sch"
+		(property "Sheetfile" "5V_5NAND/5V_5NAND.kicad_sch"
 			(at 170.7646 95.25 90)
 			(show_name no)
@@
 				(path "/13380198-0e23-4241-a844-cca11526fb8d/a0132d23-2efe-4baa-845a-d59f49944fa0"
 					(page "157")
+				)
+			)
+			(project "1_16_5V_DEMUX_NOTOUT"
+				(path "/64c295c1-a690-461e-ae3b-f66cfdb6e72a"
+					(page "14")
 				)
 			)
@@
 			)
 		)
-		(property "Sheetfile" "1_16_5V_DEMUX_NOTOUT/5V_NAND/5V_5NAND.kicad_sch"
+		(property "Sheetfile" "5V_5NAND/5V_5NAND.kicad_sch"
 			(at 117.4246 95.25 90)
 			(show_name no)
@@
 				(path "/13380198-0e23-4241-a844-cca11526fb8d/a0132d23-2efe-4baa-845a-d59f49944fa0"
 					(page "151")
+				)
+			)
+			(project "1_16_5V_DEMUX_NOTOUT"
+				(path "/64c295c1-a690-461e-ae3b-f66cfdb6e72a"
+					(page "8")
 				)
 			)
@@
 			)
 		)
-		(property "Sheetfile" "1_16_5V_DEMUX_NOTOUT/5V_NAND/5V_5NAND.kicad_sch"
+		(property "Sheetfile" "5V_5NAND/5V_5NAND.kicad_sch"
 			(at 189.8146 45.72 90)
 			(show_name no)
@@
 				(path "/13380198-0e23-4241-a844-cca11526fb8d/a0132d23-2efe-4baa-845a-d59f49944fa0"
 					(page "164")
+				)
+			)
+			(project "1_16_5V_DEMUX_NOTOUT"
+				(path "/64c295c1-a690-461e-ae3b-f66cfdb6e72a"
+					(page "17")
 				)
 			)
@@
 			)
 		)
-		(property "Sheetfile" "1_16_5V_DEMUX_NOTOUT/5V_NAND/5V_5NAND.kicad_sch"
+		(property "Sheetfile" "5V_5NAND/5V_5NAND.kicad_sch"
 			(at 152.9846 95.25 90)
 			(show_name no)
@@
 				(path "/13380198-0e23-4241-a844-cca11526fb8d/a0132d23-2efe-4baa-845a-d59f49944fa0"
 					(page "161")
+				)
+			)
+			(project "1_16_5V_DEMUX_NOTOUT"
+				(path "/64c295c1-a690-461e-ae3b-f66cfdb6e72a"
+					(page "12")
 				)
 			)
@@
 			)
 		)
-		(property "Sheetfile" "1_16_5V_DEMUX_NOTOUT/5VNOT/5VNOT.kicad_sch"
+		(property "Sheetfile" "5VNOT/5VNOT.kicad_sch"
 			(at 53.34 88.2146 0)
 			(show_name no)
@@
 				(path "/13380198-0e23-4241-a844-cca11526fb8d/a0132d23-2efe-4baa-845a-d59f49944fa0"
 					(page "148")
+				)
+			)
+			(project "1_16_5V_DEMUX_NOTOUT"
+				(path "/64c295c1-a690-461e-ae3b-f66cfdb6e72a"
+					(page "5")
 				)
 			)
@@
 			)
 		)
-		(property "Sheetfile" "1_16_5V_DEMUX_NOTOUT/5V_NAND/5V_5NAND.kicad_sch"
+		(property "Sheetfile" "5V_5NAND/5V_5NAND.kicad_sch"
 			(at 225.3746 45.72 90)
 			(show_name no)
@@
 				(path "/13380198-0e23-4241-a844-cca11526fb8d/a0132d23-2efe-4baa-845a-d59f49944fa0"
 					(page "165")
+				)
+			)
+			(project "1_16_5V_DEMUX_NOTOUT"
+				(path "/64c295c1-a690-461e-ae3b-f66cfdb6e72a"
+					(page "21")
 				)
 			)
@@
 			)
 		)
-		(property "Sheetfile" "1_16_5V_DEMUX_NOTOUT/5V_NAND/5V_5NAND.kicad_sch"
+		(property "Sheetfile" "5V_5NAND/5V_5NAND.kicad_sch"
 			(at 188.5446 95.25 90)
 			(show_name no)
@@
 				(path "/13380198-0e23-4241-a844-cca11526fb8d/a0132d23-2efe-4baa-845a-d59f49944fa0"
 					(page "158")
+				)
+			)
+			(project "1_16_5V_DEMUX_NOTOUT"
+				(path "/64c295c1-a690-461e-ae3b-f66cfdb6e72a"
+					(page "16")
 				)
 			)
@@
 			)
 		)
-		(property "Sheetfile" "1_16_5V_DEMUX_NOTOUT/5V_NAND/5V_5NAND.kicad_sch"
+		(property "Sheetfile" "5V_5NAND/5V_5NAND.kicad_sch"
 			(at 100.9146 45.72 90)
 			(show_name no)
@@
 				(path "/13380198-0e23-4241-a844-cca11526fb8d/a0132d23-2efe-4baa-845a-d59f49944fa0"
 					(page "153")
+				)
+			)
+			(project "1_16_5V_DEMUX_NOTOUT"
+				(path "/64c295c1-a690-461e-ae3b-f66cfdb6e72a"
+					(page "7")
 				)
 			)
@@
 			)
 		)
-		(property "Sheetfile" "1_16_5V_DEMUX_NOTOUT/5V_NAND/5V_5NAND.kicad_sch"
+		(property "Sheetfile" "5V_5NAND/5V_5NAND.kicad_sch"
 			(at 118.6946 45.72 90)
 			(show_name no)
@@
 				(path "/13380198-0e23-4241-a844-cca11526fb8d/a0132d23-2efe-4baa-845a-d59f49944fa0"
 					(page "154")
+				)
+			)
+			(project "1_16_5V_DEMUX_NOTOUT"
+				(path "/64c295c1-a690-461e-ae3b-f66cfdb6e72a"
+					(page "9")
 				)
 			)
@@
 			)
 		)
-		(property "Sheetfile" "1_16_5V_DEMUX_NOTOUT/5V_NAND/5V_5NAND.kicad_sch"
+		(property "Sheetfile" "5V_5NAND/5V_5NAND.kicad_sch"
 			(at 172.0346 45.72 90)
 			(show_name no)
@@
 				)
 			)
-		)
-	)
+			(project "1_16_5V_DEMUX_NOTOUT"
+				(path "/64c295c1-a690-461e-ae3b-f66cfdb6e72a"
+					(page "15")
+				)
+			)
+		)
+	)
+	(sheet_instances
+		(path "/"
+			(page "1")
+		)
+	)
