File: kicad/mainDemuxBoard/mainDemuxBoard.kicad_sch (KiCad schematic)
At the start: 16 parts, among them J1 Conn_02x20_Top_Bottom, J10 Conn_02x20_Top_Bottom, J11 Conn_02x20_Top_Bottom, J12 Conn_02x20_Top_Bottom, J13 Conn_02x20_Top_Bottom, J14 Conn_02x20_Top_Bottom, J15 Conn_02x20_Top_Bottom, J16 Conn_02x20_Top_Bottom, J2 Conn_02x20_Top_Bottom, J3 Conn_02x20_Top_Bottom, J4 Conn_02x20_Top_Bottom, J5 Conn_02x20_Top_Bottom, J6 Conn_02x20_Top_Bottom, J7 Conn_02x20_Top_Bottom, J8 Conn_02x20_Top_Bottom, J9 Conn_02x20_Top_Bottom

Commit message: finish schematic for main demux board
Parts:
- added J3: Conn_02x20_Top_Bottom, Connector_IDC:IDC-Header_2x20_P2.54mm_Latch_Vertical, symbol Connector_Generic:Conn_02x20_Top_Bottom
- J1, J15: footprint (none) -> Connector_IDC:IDC-Header_2x20_P2.54mm_Latch_Vertical
- J10: renamed from J5; footprint (none) -> Connector_IDC:IDC-Header_2x20_P2.54mm_Latch_Vertical
- J11: renamed from J13; footprint (none) -> Connector_IDC:IDC-Header_2x20_P2.54mm_Latch_Vertical
- J12: renamed from J6; footprint (none) -> Connector_IDC:IDC-Header_2x20_P2.54mm_Latch_Vertical
- J13: renamed from J14; footprint (none) -> Connector_IDC:IDC-Header_2x20_P2.54mm_Latch_Vertical
- J14: renamed from J7; footprint (none) -> Connector_IDC:IDC-Header_2x20_P2.54mm_Latch_Vertical
- J16: renamed from J8; footprint (none) -> Connector_IDC:IDC-Header_2x20_P2.54mm_Latch_Vertical
- J17: renamed from J16; footprint (none) -> Connector_IDC:IDC-Header_2x20_P2.54mm_Latch_Vertical
- J2: renamed from J9; footprint (none) -> Connector_IDC:IDC-Header_2x20_P2.54mm_Latch_Vertical
- J4: renamed from J2; footprint (none) -> Connector_IDC:IDC-Header_2x20_P2.54mm_Latch_Vertical
- J5: renamed from J10; footprint (none) -> Connector_IDC:IDC-Header_2x20_P2.54mm_Latch_Vertical
- J6: renamed from J3; footprint (none) -> Connector_IDC:IDC-Header_2x20_P2.54mm_Latch_Vertical
- J7: renamed from J11; footprint (none) -> Connector_IDC:IDC-Header_2x20_P2.54mm_Latch_Vertical
- J8: renamed from J4; footprint (none) -> Connector_IDC:IDC-Header_2x20_P2.54mm_Latch_Vertical
- J9: renamed from J12; footprint (none) -> Connector_IDC:IDC-Header_2x20_P2.54mm_Latch_Vertical
Connections:
- net +10V: now also J3.10 (Pin_10), J3.11 (Pin_11), J3.12 (Pin_12)
- net +5V: now also J3.13 (Pin_13), J3.14 (Pin_14), J3.15 (Pin_15), J3.16 (Pin_16), J3.17 (Pin_17)
- net BL_{0}: now also J3.21 (Pin_21)
- net BL_{1}: now also J3.23 (Pin_23)
- net BL_{2}: now also J3.25 (Pin_25)
- net BL_{3}: now also J3.27 (Pin_27)
- net BL_{4}: now also J3.29 (Pin_29)
- net BL_{5}: now also J3.31 (Pin_31)
- net BL_{6}: now also J3.33 (Pin_33)
- net BL_{7}: now also J3.35 (Pin_35)
- net GND: now also J3.18 (Pin_18), J3.19 (Pin_19), J3.20 (Pin_20), J3.37 (Pin_37), J3.38 (Pin_38), J3.39 (Pin_39), J3.40 (Pin_40)
- net S_{0}: now also J3.1 (Pin_1)
- net S_{1}: now also J3.2 (Pin_2)
- net S_{2}: now also J3.3 (Pin_3)
- net S_{3}: now also J3.4 (Pin_4)
- net ~{BL_{0}}: now also J3.22 (Pin_22)
- net ~{BL_{1}}: now also J3.24 (Pin_24)
- net ~{BL_{2}}: now also J3.26 (Pin_26)
- net ~{BL_{3}}: now also J3.28 (Pin_28)
- net ~{BL_{4}}: now also J3.30 (Pin_30)
- net ~{BL_{5}}: now also J3.32 (Pin_32)
- net ~{BL_{6}}: now also J3.34 (Pin_34)
- net ~{BL_{7}}: now also J3.36 (Pin_36)
- net A_{15}: now reaches J17.5 (Pin_5)
- net A_{9}: now reaches J5.5 (Pin_5)
- net A_{4}: now reaches J10.5 (Pin_5)
- net A_{13}: now reaches J13.5 (Pin_5)
- net A_{7}: now reaches J16.5 (Pin_5)
- net A_{12}: now reaches J11.5 (Pin_5)
- net A_{10}: now reaches J7.5 (Pin_5)
- net A_{14}: now reaches J15.5 (Pin_5)
- net A_{8}: now reaches J2.5 (Pin_5)
- net A_{3}: now reaches J8.5 (Pin_5)
- net A_{11}: now reaches J9.5 (Pin_5)
- net A_{0}: now reaches J1.5 (Pin_5)
- net A_{5}: now reaches J12.5 (Pin_5)
- net A_{6}: now reaches J14.5 (Pin_5)
- net A_{1}: now reaches J4.5 (Pin_5)
- net A_{2}: now reaches J6.5 (Pin_5)
- new net 1_16_5V_DEMUX_NOTOUT/D: J3.9 (Pin_9)
- new net 1_16_5V_DEMUX_NOTOUT/S_{0}: J3.5 (Pin_5)
- new net 1_16_5V_DEMUX_NOTOUT/S_{1}: J3.6 (Pin_6)
- new net 1_16_5V_DEMUX_NOTOUT/S_{2}: J3.7 (Pin_7)
- new net 1_16_5V_DEMUX_NOTOUT/S_{3}: J3.8 (Pin_8)
Other:
- added sheet 16_NOT (16_NOT/16_NOT.kicad_sch)
- added sheet 1_16_5V_DEMUX_NOTOUT (1_16_5V_DEMUX_NOTOUT/1_16_5V_DEMUX_NOTOUT.kicad_sch)
