File: kicad/controllerBoard/controllerBoard.kicad_sch (KiCad schematic)
At the start: 19 parts, among them J1 Conn_02x20_Top_Bottom, J2 Conn_02x20_Top_Bottom, Q635 WTM30N02VD, U1 LM3478MA

Commit message: did stuff
Parts:
- renumbered C14 to C1, C11 to C2, C13 to C3, C10 to C4, C9 to C5, C12 to C6, D5 to D1, D6 to D2, Q635 to Q1, R52 to R1, R51 to R2, R50 to R3, R49 to R4, R53 to R5, R54 to R6
Changed lines of the file:
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@@
 		(dnp no)
 		(fields_autoplaced yes)
-		(property "Reference" "#PWR094"
+		(property "Reference" "#PWR07"
 			(at 115.57 153.67 0)
 			(hide yes)
@@
 			(project "controllerBoard"
 				(path "/93a9a1ca-4ee5-40da-ab67-92836146c003"
-					(reference "#PWR094")
+					(reference "#PWR07")
 					(unit 1)
 				)
@@
 		(dnp no)
 		(fields_autoplaced yes)
-		(property "Reference" "C12"
+		(property "Reference" "C6"
 			(at 119.38 170.1799 0)
 			(show_name no)
@@
 			(project "controllerBoard"
 				(path "/93a9a1ca-4ee5-40da-ab67-92836146c003"
-					(reference "C12")
+					(reference "C6")
 					(unit 1)
 				)
@@
 		(dnp no)
 		(fields_autoplaced yes)
-		(property "Reference" "R53"
+		(property "Reference" "R5"
 			(at 109.22 156.2099 0)
 			(show_name no)
@@
 			(project "controllerBoard"
 				(path "/93a9a1ca-4ee5-40da-ab67-92836146c003"
-					(reference "R53")
+					(reference "R5")
 					(unit 1)
 				)
@@
 		(dnp no)
 		(fields_autoplaced yes)
-		(property "Reference" "#PWR03"
+		(property "Reference" "#PWR05"
 			(at 38.1 83.82 0)
 			(hide yes)
@@
 			(project "controllerBoard"
 				(path "/93a9a1ca-4ee5-40da-ab67-92836146c003"
-					(reference "#PWR03")
+					(reference "#PWR05")
 					(unit 1)
 				)
@@
 		(dnp no)
 		(fields_autoplaced yes)
-		(property "Reference" "R54"
+		(property "Reference" "R6"
 			(at 109.22 177.7999 0)
 			(show_name no)
@@
 			(project "controllerBoard"
 				(path "/93a9a1ca-4ee5-40da-ab67-92836146c003"
-					(reference "R54")
+					(reference "R6")
 					(unit 1)
 				)
@@
 		(dnp no)
 		(fields_autoplaced yes)
-		(property "Reference" "D6"
+		(property "Reference" "D2"
 			(at 124.46 152.3999 90)
 			(show_name no)
@@
 			(project "controllerBoard"
 				(path "/93a9a1ca-4ee5-40da-ab67-92836146c003"
-					(reference "D6")
+					(reference "D2")
 					(unit 1)
 				)
@@
 		(dnp no)
 		(fields_autoplaced yes)
-		(property "Reference" "C14"
+		(property "Reference" "C1"
 			(at 34.29 152.3999 0)
 			(show_name no)
@@
 			(project "controllerBoard"
 				(path "/93a9a1ca-4ee5-40da-ab67-92836146c003"
-					(reference "C14")
+					(reference "C1")
 					(unit 1)
 				)
@@
 		(dnp no)
 		(fields_autoplaced yes)
-		(property "Reference" "#PWR093"
+		(property "Reference" "#PWR06"
 			(at 66.04 189.23 0)
 			(hide yes)
@@
 			(project "controllerBoard"
 				(path "/93a9a1ca-4ee5-40da-ab67-92836146c003"
-					(reference "#PWR093")
+					(reference "#PWR06")
 					(unit 1)
 				)
@@
 		(dnp no)
 		(fields_autoplaced yes)
-		(property "Reference" "C11"
+		(property "Reference" "C2"
 			(at 41.91 177.7999 0)
 			(show_name no)
@@
 			(project "controllerBoard"
 				(path "/93a9a1ca-4ee5-40da-ab67-92836146c003"
-					(reference "C11")
+					(reference "C2")
 					(unit 1)
 				)
@@
 		(dnp no)
 		(fields_autoplaced yes)
-		(property "Reference" "R49"
+		(property "Reference" "R4"
 			(at 99.06 177.7999 0)
 			(show_name no)
@@
 			(project "controllerBoard"
 				(path "/93a9a1ca-4ee5-40da-ab67-92836146c003"
-					(reference "R49")
+					(reference "R4")
 					(unit 1)
 				)
@@
 		(dnp no)
 		(fields_autoplaced yes)
-		(property "Reference" "#PWR0112"
+		(property "Reference" "#PWR03"
 			(at 36.83 153.67 0)
 			(hide yes)
@@
 			(project "controllerBoard"
 				(path "/93a9a1ca-4ee5-40da-ab67-92836146c003"
-					(reference "#PWR0112")
+					(reference "#PWR03")
 					(unit 1)
 				)
@@
 		(dnp no)
 		(fields_autoplaced yes)
-		(property "Reference" "Q635"
+		(property "Reference" "Q1"
 			(at 100.33 161.2899 0)
 			(show_name no)
@@
 			(project "controllerBoard"
 				(path "/93a9a1ca-4ee5-40da-ab67-92836146c003"
-					(reference "Q635")
+					(reference "Q1")
 					(unit 1)
 				)
@@
 		(dnp no)
 		(fields_autoplaced yes)
-		(property "Reference" "#PWR0111"
+		(property "Reference" "#PWR08"
 			(at 121.92 163.83 0)
 			(hide yes)
@@
 			(project "controllerBoard"
 				(path "/93a9a1ca-4ee5-40da-ab67-92836146c003"
-					(reference "#PWR0111")
+					(reference "#PWR08")
 					(unit 1)
 				)
@@
 		(dnp no)
 		(fields_autoplaced yes)
-		(property "Reference" "D5"
+		(property "Reference" "D1"
 			(at 100.33 143.51 0)
 			(show_name no)
@@
 			(project "controllerBoard"
 				(path "/93a9a1ca-4ee5-40da-ab67-92836146c003"
-					(reference "D5")
+					(reference "D1")
 					(unit 1)
 				)
@@
 		(dnp no)
 		(fields_autoplaced yes)
-		(property "Reference" "R51"
+		(property "Reference" "R2"
 			(at 50.8 177.7999 0)
 			(show_name no)
@@
 			(project "controllerBoard"
 				(path "/93a9a1ca-4ee5-40da-ab67-92836146c003"
-					(reference "R51")
+					(reference "R2")
 					(unit 1)
 				)
@@
 		(dnp no)
 		(fields_autoplaced yes)
-		(property "Reference" "C13"
+		(property "Reference" "C3"
 			(at 45.72 152.3999 0)
 			(show_name no)
@@
 			(project "controllerBoard"
 				(path "/93a9a1ca-4ee5-40da-ab67-92836146c003"
-					(reference "C13")
+					(reference "C3")
 					(unit 1)
 				)
@@
 		(dnp no)
 		(fields_autoplaced yes)
-		(property "Reference" "R52"
+		(property "Reference" "R1"
 			(at 34.29 167.6399 0)
 			(show_name no)
@@
 			(project "controllerBoard"
 				(path "/93a9a1ca-4ee5-40da-ab67-92836146c003"
-					(reference "R52")
+					(reference "R1")
 					(unit 1)
 				)
@@
 		(dnp no)
 		(fields_autoplaced yes)
-		(property "Reference" "C10"
+		(property "Reference" "C4"
 			(at 52.07 170.1799 0)
 			(show_name no)
@@
 			(project "controllerBoard"
 				(path "/93a9a1ca-4ee5-40da-ab67-92836146c003"
-					(reference "C10")
+					(reference "C4")
 					(unit 1)
 				)
@@
 		(dnp no)
 		(fields_autoplaced yes)
-		(property "Reference" "R50"
+		(property "Reference" "R3"
 			(at 88.9 165.1 90)
 			(show_name no)
@@
 			(project "controllerBoard"
 				(path "/93a9a1ca-4ee5-40da-ab67-92836146c003"
-					(reference "R50")
+					(reference "R3")
 					(unit 1)
 				)
@@
 		(dnp no)
 		(fields_autoplaced yes)
-		(property "Reference" "#PWR095"
+		(property "Reference" "#PWR04"
 			(at 36.83 163.83 0)
 			(hide yes)
@@
 			(project "controllerBoard"
 				(path "/93a9a1ca-4ee5-40da-ab67-92836146c003"
-					(reference "#PWR095")
+					(reference "#PWR04")
 					(unit 1)
 				)
@@
 		(dnp no)
 		(fields_autoplaced yes)
-		(property "Reference" "C9"
+		(property "Reference" "C5"
 			(at 88.9 177.7999 0)
 			(show_name no)
@@
 			(project "controllerBoard"
 				(path "/93a9a1ca-4ee5-40da-ab67-92836146c003"
-					(reference "C9")
-					(unit 1)
-				)
+					(reference "C5")
+					(unit 1)
+				)

Commit message: change to charge pump
Parts:
- removed C1: 470uC, symbol Device:C
- removed C2: 15nC, symbol Device:C
- removed C3: 100nC, symbol Device:C
- removed C4: 330nC, symbol Device:C
- removed C5: 10pC, symbol Device:C
- removed C6: 180uC, symbol Device:C
- removed D1: D, symbol Device:D
- removed D2: SMBJ5348B, symbol Device:D_Zener
- removed L1: 15uL, symbol Device:L
- removed Q1: WTM30N02VD, symbol Simulation_SPICE:NMOS
- removed R1: 133kR, symbol Device:R
- removed R2, R6: 1kR, symbol Device:R
- removed R3: 100R, symbol Device:R
- removed R4: 12mR, symbol Device:R
- removed R5: 6.98kR, symbol Device:R
- removed U1: LM3478MA, Package_SO:SOIC-8_3.9x4.9mm_P1.27mm, symbol Regulator_Controller:LM3478MA
- added C15: 47uC, symbol Device:C
- added C16: 100nC, symbol Device:C
Connections:
- net +5V: now also C15.1, C16.1
- net GND: now also C15.2, C16.2
Other:
- added sheet 5V_TO_10V (5V_TO_10V\5V_TO_10V.kicad_sch)

Commit message: did more simulation, added bom
Parts:
- renumbered C15 to C1, C16 to C2
Other:
- sheet 5V_TO_10V: file 5V_TO_10V\5V_TO_10V.kicad_sch -> 5V_TO_10V/5V_TO_10V.kicad_sch
Changed lines of the file:
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@@
 	(rectangle
 		(start 16.51 133.35)
-		(end 142.24 194.31)
+		(end 95.25 176.53)
 		(stroke
 			(width 0)
@@
 		(dnp no)
 		(fields_autoplaced yes)
-		(property "Reference" "C16"
+		(property "Reference" "C2"
 			(at 43.18 156.2099 0)
 			(show_name no)
@@
 			(project "controllerBoard"
 				(path "/93a9a1ca-4ee5-40da-ab67-92836146c003"
-					(reference "C16")
+					(reference "C2")
 					(unit 1)
 				)
@@
 		(dnp no)
 		(fields_autoplaced yes)
-		(property "Reference" "C15"
+		(property "Reference" "C1"
 			(at 25.4 156.2099 0)
 			(show_name no)
@@
 			(project "controllerBoard"
 				(path "/93a9a1ca-4ee5-40da-ab67-92836146c003"
-					(reference "C15")
+					(reference "C1")
 					(unit 1)
 				)
@@
 		(dnp no)
 		(fields_autoplaced yes)
-		(property "Reference" "#PWR0134"
+		(property "Reference" "#PWR06"
 			(at 77.47 163.83 0)
 			(hide yes)
@@
 			(project "controllerBoard"
 				(path "/93a9a1ca-4ee5-40da-ab67-92836146c003"
-					(reference "#PWR0134")
+					(reference "#PWR06")
 					(unit 1)
 				)
@@
 		(dnp no)
 		(fields_autoplaced yes)
-		(property "Reference" "#PWR0135"
+		(property "Reference" "#PWR03"
 			(at 30.48 157.48 0)
 			(hide yes)
@@
 			(project "controllerBoard"
 				(path "/93a9a1ca-4ee5-40da-ab67-92836146c003"
-					(reference "#PWR0135")
+					(reference "#PWR03")
 					(unit 1)
 				)
@@
 		(dnp no)
 		(fields_autoplaced yes)
-		(property "Reference" "#PWR0136"
+		(property "Reference" "#PWR04"
 			(at 30.48 167.64 0)
 			(hide yes)
@@
 			(project "controllerBoard"
 				(path "/93a9a1ca-4ee5-40da-ab67-92836146c003"
-					(reference "#PWR0136")
+					(reference "#PWR04")
 					(unit 1)
 				)
@@
 			)
 		)
-		(property "Sheetfile" "5V_TO_10V\\5V_TO_10V.kicad_sch"
+		(property "Sheetfile" "5V_TO_10V/5V_TO_10V.kicad_sch"
 			(at 54.61 168.2246 0)
 			(show_name no)
