File: kicad/controllerBoard/controllerBoard.kicad_pcb (KiCad board)
At the start: 2 copper layers, 739 parts, among them J1 Conn_02x20_Top_Bottom, J2 Conn_02x20_Top_Bottom, Q1 Q_PMOS_GSD, Q10 Q_NMOS_GSD, Q100 Q_NMOS_GSD, Q101 Q_PMOS_GSD, Q102 Q_NMOS_GSD, Q103 Q_PMOS_GSD, Q104 Q_NMOS_GSD, Q105 Q_PMOS_GSD, Q106 Q_NMOS_GSD, Q107 Q_PMOS_GSD, Q108 Q_NMOS_GSD, Q109 Q_PMOS_GSD, Q11 Q_PMOS_GSD, Q110 Q_NMOS_GSD, Q111 Q_PMOS_GSD, Q112 Q_NMOS_GSD, Q113 Q_PMOS_GSD, Q114 Q_NMOS_GSD, Q115 Q_PMOS_GSD, Q116 Q_NMOS_GSD, Q117 Q_PMOS_GSD, Q118 Q_NMOS_GSD, Q119 Q_PMOS_GSD, Q12 Q_NMOS_GSD, Q120 Q_NMOS_GSD, Q121 Q_PMOS_GSD, Q122 Q_NMOS_GSD, Q123 Q_PMOS_GSD, Q124 Q_NMOS_GSD, Q125 Q_PMOS_GSD, Q126 Q_NMOS_GSD, Q127 Q_PMOS_GSD, Q128 Q_NMOS_GSD, Q129 Q_PMOS_GSD, Q13 Q_PMOS_GSD, Q130 Q_NMOS_GSD, Q131 Q_PMOS_GSD, Q132 Q_NMOS_GSD, Q133 Q_PMOS_GSD, Q134 Q_NMOS_GSD, Q135 Q_PMOS_GSD, Q136 Q_NMOS_GSD, Q137 Q_PMOS_GSD, Q138 Q_NMOS_GSD, Q139 Q_PMOS_GSD, Q14 Q_PMOS_GSD, Q140 Q_NMOS_GSD, Q141 Q_PMOS_GSD, Q142 Q_NMOS_GSD, Q143 Q_PMOS_GSD, Q144 Q_NMOS_GSD, Q145 Q_PMOS_GSD, Q146 Q_NMOS_GSD, Q147 Q_PMOS_GSD, Q148 Q_NMOS_GSD, Q149 Q_PMOS_GSD, Q15 Q_PMOS_GSD, Q150 Q_NMOS_GSD, Q151 Q_PMOS_GSD, Q152 Q_NMOS_GSD, Q153 Q_PMOS_GSD, Q154 Q_NMOS_GSD, Q155 Q_PMOS_GSD, Q156 Q_NMOS_GSD, Q157 Q_PMOS_GSD, Q158 Q_NMOS_GSD, Q159 Q_PMOS_GSD, Q16 Q_NMOS_GSD, Q160 Q_NMOS_GSD, Q161 Q_PMOS_GSD, Q162 Q_NMOS_GSD, Q163 Q_PMOS_GSD, Q164 Q_NMOS_GSD, Q165 Q_PMOS_GSD, Q166 Q_NMOS_GSD, Q167 Q_PMOS_GSD, Q168 Q_NMOS_GSD, Q169 Q_PMOS_GSD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

Commit message: finished routing all sub schematics
Parts:
- removed C1: 47uC, Capacitor_SMD:C_1206_3216Metric
- removed C2: 100nC, Capacitor_SMD:C_0805_2012Metric
- added C17: 100nC, Capacitor_SMD:C_0805_2012Metric, F.Cu at (60.2, 19.4)
- added C18: 100nC, Capacitor_SMD:C_0805_2012Metric, F.Cu at (62.1, 56.4)
- added C19: 100nC, Capacitor_SMD:C_0805_2012Metric, F.Cu at (52.1, 20.4)
- added C20: 100nC, Capacitor_SMD:C_0805_2012Metric, F.Cu at (50.9, 56.6)
- added C21: 100nC, Capacitor_SMD:C_0805_2012Metric, F.Cu at (51.0, 30.3)
- added C22: 100nC, Capacitor_SMD:C_0805_2012Metric, F.Cu at (62.9, 32.4)
- added C23: 100nC, Capacitor_SMD:C_0805_2012Metric, F.Cu at (61.7, 44.2)
- added C24: 100nC, Capacitor_SMD:C_0805_2012Metric, F.Cu at (50.4, 43.1)
- added C25: 100nC, Capacitor_SMD:C_0805_2012Metric, F.Cu at (53.7, 31.4)
- added C26: C_Polarized, Capacitor_THT:CP_Radial_D10.0mm_P5.00mm, F.Cu at (46.1, 34.5)
- added C27: C_Polarized, Capacitor_THT:CP_Radial_D10.0mm_P5.00mm, F.Cu at (67.3, 47.3)
- added C28: C_Polarized, Capacitor_THT:CP_Radial_D10.0mm_P5.00mm, F.Cu at (46.9, 47.2)
- added C29: C_Polarized, Capacitor_THT:CP_Radial_D10.0mm_P5.00mm, F.Cu at (67.4, 36.2)
- added C30: C_Polarized, Capacitor_THT:CP_Radial_D10.0mm_P5.00mm, F.Cu at (57.6, 65.8)
- added Q649: Q_PMOS_GSD, easyeda2kicad:SOT-23-P, F.Cu at (58.4, 55.4)
- added Q650: Q_NMOS_GSD, easyeda2kicad:SOT-23-N, F.Cu at (54.7, 55.3)
- added Q651: Q_PMOS_GSD, easyeda2kicad:SOT-23-P, F.Cu at (58.4, 51.4)
- added Q652: Q_NMOS_GSD, easyeda2kicad:SOT-23-N, F.Cu at (54.7, 51.3)
- C12, C14, C15, C16: value 1mC -> 100nC; footprint Capacitor_THT:CP_Radial_D10.0mm_P5.00mm -> Capacitor_SMD:C_0805_2012Metric
- C13: value 1mC -> 4.7uC; footprint Capacitor_THT:CP_Radial_D10.0mm_P5.00mm -> Capacitor_SMD:C_0805_2012Metric
- C6, C9: value 4.7uC -> 100nC
- C8: value 100nC -> 4.7uC
- moved C10 149.8 mm to (81.5, 155.5)
- moved Q387 148.0 mm to (47.3, 159.7)
- moved Q388 147.2 mm to (47.3, 163.2)
- moved Q389 147.1 mm to (54.0, 159.6)
- moved Q390 146.4 mm to (54.1, 163.2)
- moved Q497 146.3 mm to (145.6, 39.5)
- moved Q617 144.7 mm to (104.3, 158.4)
- moved Q391 144.4 mm to (60.1, 157.1)
- moved Q618 144.0 mm to (104.2, 162.0)
- moved Q619 143.9 mm to (111.0, 158.3)
- moved Q392 143.5 mm to (60.4, 160.7)
- moved Q500 143.4 mm to (148.5, 41.6)
- moved Q499 143.3 mm to (148.4, 37.3)
- moved Q620 143.1 mm to (111.0, 161.9)
- moved R45 143.0 mm to (40.1, 152.3), turned to -90 degrees
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Connections:
- C10 pad 1: Net-(Q616-D) -> GND
- C10 pad 2: Net-(D4-K) -> +5V
- C11 pad 1: Net-(Q635-G) -> /WL_PULSE
- C11 pad 2: GND -> Net-(D3-K)
- C12 pad 1: Net-(D6-K) -> GND
- C12 pad 2: Net-(Q641-D) -> Net-(Q415-G)
- C13 pad 1: Net-(D5-K) -> GND
- C13 pad 2: Net-(Q645-D) -> Net-(Q416-D)
- C14 pad 1: Net-(D10-A) -> Net-(Q616-D)
- C14 pad 2: Net-(Q645-D) -> Net-(D4-K)
- C15 pad 1: Net-(D7-K) -> GND
- C15 pad 2: Net-(Q641-D) -> +5V
- C16 pad 1: +10V -> GND
- C16 pad 2: GND -> +5V
- C4 pad 1: /~{EN_{input}} -> GND
- C4 pad 2: Net-(D2-K) -> +5V
- C5 pad 2: Net-(Q407-G) -> +5V
- C6 pad 1: GND -> /~{EN_{input}}
- C6 pad 2: Net-(Q408-D) -> Net-(D2-K)
- C7 pad 1: /WL_PULSE -> GND
- C7 pad 2: Net-(D3-K) -> Net-(Q407-G)
- C8 pad 2: Net-(Q415-G) -> Net-(Q408-D)
- C9 pad 2: Net-(Q416-D) -> +5V
- Q645 pad 1: Net-(Q641-D) -> Net-(Q639-G)
- Q645 pad 3: Net-(Q645-D) -> Net-(Q641-D)
- Q646 pad 1: Net-(Q641-D) -> Net-(Q639-G)
- Q646 pad 3: Net-(Q645-D) -> Net-(Q641-D)
- Q647 pad 3: Net-(Q645-D) -> Net-(Q647-D)
- Q648 pad 3: Net-(Q645-D) -> Net-(Q647-D)
Routing:
- net /~{EN_{input}}: track 0.00 -> 709.1 mm, vias 0 -> 50
- net /EN_{input}: track 0.00 -> 696.8 mm
- net /8DLATCH4/~{EN}: track 0.00 -> 237.2 mm, vias 0 -> 16
- net /OP_{in}: track 0.00 -> 235.6 mm
- net /R_PULSE: track 0.00 -> 235.3 mm
- net /~{R_PULSE}: track 0.00 -> 230.0 mm, vias 0 -> 16
- net /8DLATCH4/EN: track 0.00 -> 227.1 mm
- net +5V: track 0.00 -> 188.9 mm, vias 0 -> 90
- net GND: track 0.00 -> 180.8 mm, vias 0 -> 75
- net +10V: track 0.00 -> 85.2 mm
- net Net-(Q641-D): track 0.00 -> 70.1 mm, vias 0 -> 3
- net Net-(Q639-G): track 0.00 -> 58.5 mm, vias 0 -> 4
- net Net-(Q647-D): track 0.00 -> 37.5 mm
- net /CLK: track 0.00 -> 29.0 mm
- net Net-(D10-A): track 0.00 -> 27.6 mm
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Other:
- board outline added: 150 x 150 mm
