File: kicad/mainDemuxBoard/1_16_5V_DEMUX_NOTOUT/5VNOT/5VNOT.kicad_sch (KiCad schematic)
At the start: 2 parts, among them Q1 PMOS, Q2 NMOS

Commit message: finish main demux board
Parts:
- renumbered Q1 to Q3, Q2 to Q4
Changed lines of the file:
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@@
 		(dnp no)
 		(fields_autoplaced yes)
-		(property "Reference" "Q2"
+		(property "Reference" "Q4"
 			(at 120.65 68.5799 0)
 			(show_name no)
@@
 		(dnp no)
 		(fields_autoplaced yes)
-		(property "Reference" "#PWR052"
+		(property "Reference" "#PWR054"
 			(at 116.84 53.34 0)
 			(hide yes)
@@
 		(dnp no)
 		(fields_autoplaced yes)
-		(property "Reference" "Q1"
+		(property "Reference" "Q3"
 			(at 120.65 53.3399 0)
 			(show_name no)
@@
 		(dnp no)
 		(fields_autoplaced yes)
-		(property "Reference" "#PWR053"
+		(property "Reference" "#PWR055"
 			(at 116.84 81.28 0)
 			(hide yes)

Commit message: update main board schematic
Parts:
- Q1: renamed from Q3; value PMOS -> Q_PMOS_GSD; symbol Simulation_SPICE:PMOS -> Transistor_FET:Q_PMOS_GSD
- Q2: renamed from Q4; value NMOS -> Q_NMOS_GSD; symbol Simulation_SPICE:NMOS -> Transistor_FET:Q_NMOS_GSD
Connections:
- net +5V: now also Q1.2 (S); no longer Q1.3 (S)
- net A: now also Q1.1 (G), Q2.1 (G); no longer Q1.2 (G), Q2.2 (G)
- net GND: now also Q2.2 (S); no longer Q2.3 (S)
- net Y: now also Q1.3 (D), Q2.3 (D); no longer Q1.1 (D), Q2.1 (D)
Changed lines of the file:
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@@
 	)
 	(symbol
-		(lib_id "Simulation_SPICE:NMOS")
+		(lib_id "Transistor_FET:Q_NMOS_GSD")
 		(at 114.3 69.85 0)
 		(unit 1)
@@
 		(dnp no)
 		(fields_autoplaced yes)
-		(property "Reference" "Q4"
+		(property "Reference" "Q2"
 			(at 120.65 68.5799 0)
 			(show_name no)
@@
 			)
 		)
-		(property "Value" "NMOS"
+		(property "Value" "Q_NMOS_GSD"
 			(at 120.65 71.1199 0)
 			(show_name no)
@@
 				(path "/64c295c1-a690-461e-ae3b-f66cfdb6e72a/afd2047a-5605-416e-9801-fddbd3089131"
 					(reference "Q8")
+					(unit 1)
+				)
+			)
+			(project "5VNOT"
+				(path "/cabc387a-6207-4601-83a6-292a0d885e49"
+					(reference "Q1160")
 					(unit 1)
 				)
@@
 		(dnp no)
 		(fields_autoplaced yes)
-		(property "Reference" "#PWR054"
+		(property "Reference" "#PWR052"
 			(at 116.84 53.34 0)
 			(hide yes)
@@
 			(project "sramBoard"
 				(path "/13380198-0e23-4241-a844-cca11526fb8d/a0132d23-2efe-4baa-845a-d59f49944fa0/0600d891-ccd3-4602-9849-fea3d7e045ca"
-					(reference "#PWR0522")
+					(reference "#PWR0654")
 					(unit 1)
 				)
 				(path "/13380198-0e23-4241-a844-cca11526fb8d/a0132d23-2efe-4baa-845a-d59f49944fa0/2e151ebf-7913-49eb-83f7-10f1b73fc84d"
-					(reference "#PWR0520")
+					(reference "#PWR0652")
 					(unit 1)
 				)
 				(path "/13380198-0e23-4241-a844-cca11526fb8d/a0132d23-2efe-4baa-845a-d59f49944fa0/40364bbe-d9b2-4f0d-a83e-984d8754432c"
-					(reference "#PWR0516")
+					(reference "#PWR0648")
 					(unit 1)
 				)
 				(path "/13380198-0e23-4241-a844-cca11526fb8d/a0132d23-2efe-4baa-845a-d59f49944fa0/afd2047a-5605-416e-9801-fddbd3089131"
-					(reference "#PWR0518")
+					(reference "#PWR0650")
 					(unit 1)
 				)
@@
 				)
 			)
+			(project "5VNOT"
+				(path "/cabc387a-6207-4601-83a6-292a0d885e49"
+					(reference "#PWR0522")
+					(unit 1)
+				)
+			)
 			(project "mainDemuxBoard"
 				(path "/f888c822-9b6b-4788-a884-52437644ebdc/1a45d35c-9d3b-4677-823d-3f805a376771/0600d891-ccd3-4602-9849-fea3d7e045ca"
@@
 	)
 	(symbol
-		(lib_id "Simulation_SPICE:PMOS")
+		(lib_id "Transistor_FET:Q_PMOS_GSD")
 		(at 114.3 54.61 0)
 		(mirror x)
@@
 		(dnp no)
 		(fields_autoplaced yes)
-		(property "Reference" "Q3"
+		(property "Reference" "Q1"
 			(at 120.65 53.3399 0)
 			(show_name no)
@@
 			)
 		)
-		(property "Value" "PMOS"
+		(property "Value" "Q_PMOS_GSD"
 			(at 120.65 55.8799 0)
 			(show_name no)
@@
 				(path "/64c295c1-a690-461e-ae3b-f66cfdb6e72a/afd2047a-5605-416e-9801-fddbd3089131"
 					(reference "Q7")
+					(unit 1)
+				)
+			)
+			(project "5VNOT"
+				(path "/cabc387a-6207-4601-83a6-292a0d885e49"
+					(reference "Q1159")
 					(unit 1)
 				)
@@
 		(dnp no)
 		(fields_autoplaced yes)
-		(property "Reference" "#PWR055"
+		(property "Reference" "#PWR053"
 			(at 116.84 81.28 0)
 			(hide yes)
@@
 			(project "sramBoard"
 				(path "/13380198-0e23-4241-a844-cca11526fb8d/a0132d23-2efe-4baa-845a-d59f49944fa0/0600d891-ccd3-4602-9849-fea3d7e045ca"
-					(reference "#PWR0523")
+					(reference "#PWR0655")
 					(unit 1)
 				)
 				(path "/13380198-0e23-4241-a844-cca11526fb8d/a0132d23-2efe-4baa-845a-d59f49944fa0/2e151ebf-7913-49eb-83f7-10f1b73fc84d"
-					(reference "#PWR0521")
+					(reference "#PWR0653")
 					(unit 1)
 				)
 				(path "/13380198-0e23-4241-a844-cca11526fb8d/a0132d23-2efe-4baa-845a-d59f49944fa0/40364bbe-d9b2-4f0d-a83e-984d8754432c"
-					(reference "#PWR0517")
+					(reference "#PWR0649")
 					(unit 1)
 				)
 				(path "/13380198-0e23-4241-a844-cca11526fb8d/a0132d23-2efe-4baa-845a-d59f49944fa0/afd2047a-5605-416e-9801-fddbd3089131"
-					(reference "#PWR0519")
+					(reference "#PWR0651")
 					(unit 1)
 				)
@@
 				)
 			)
+			(project "5VNOT"
+				(path "/cabc387a-6207-4601-83a6-292a0d885e49"
+					(reference "#PWR0523")
+					(unit 1)
+				)
+			)
 			(project "mainDemuxBoard"
 				(path "/f888c822-9b6b-4788-a884-52437644ebdc/1a45d35c-9d3b-4677-823d-3f805a376771/0600d891-ccd3-4602-9849-fea3d7e045ca"
@@
 		)
 	)
+	(sheet_instances
+		(path "/"
+			(page "1")
+		)
+	)
