File: kicad/mainDemuxBoard/1_16_5V_DEMUX_NOTOUT/5V_5NAND/5V_5NAND.kicad_sch (KiCad schematic)
At the start: 10 parts, among them Q10 PMOS, Q11 PMOS, Q12 PMOS, Q13 PMOS, Q14 NMOS, Q15 NMOS, Q16 NMOS, Q17 NMOS, Q18 NMOS, Q9 PMOS

Commit message: update main board schematic
Parts:
- Q10, Q11, Q12, Q13, Q9: value PMOS -> Q_PMOS_GSD; symbol Simulation_SPICE:PMOS -> Transistor_FET:Q_PMOS_GSD
- Q14, Q15, Q16, Q17, Q18: value NMOS -> Q_NMOS_GSD; symbol Simulation_SPICE:NMOS -> Transistor_FET:Q_NMOS_GSD
Connections:
- net +5V: now also Q10.2 (S), Q11.2 (S), Q12.2 (S), Q13.2 (S), Q9.2 (S); no longer Q10.3 (S), Q11.3 (S), Q12.3 (S), Q13.3 (S), Q9.3 (S)
- net A_{0}: now also Q13.1 (G), Q14.1 (G); no longer Q13.2 (G), Q14.2 (G)
- net A_{1}: now also Q12.1 (G), Q15.1 (G); no longer Q12.2 (G), Q15.2 (G)
- net A_{2}: now also Q11.1 (G), Q16.1 (G); no longer Q11.2 (G), Q16.2 (G)
- net A_{3}: now also Q10.1 (G), Q17.1 (G); no longer Q10.2 (G), Q17.2 (G)
- net A_{4}: now also Q18.1 (G), Q9.1 (G); no longer Q18.2 (G), Q9.2 (G)
- net GND: now also Q18.2 (S); no longer Q18.3 (S)
- net Y: now also Q10.3 (D), Q11.3 (D), Q12.3 (D), Q13.3 (D), Q14.3 (D), Q9.3 (D); no longer Q10.1 (D), Q11.1 (D), Q12.1 (D), Q13.1 (D), Q14.1 (D), Q9.1 (D)
- net at Q15.3 (D): now also Q14.2 (S); no longer Q16.1 (D)
- net at Q16.3 (D): now also Q15.2 (S); no longer Q17.1 (D)
- net at Q17.3 (D): now also Q16.2 (S); no longer Q18.1 (D)
- new net: Q17.2 (S), Q18.3 (D)
