File: kicad/controllerBoard/8DLATCH/8DLATCH.kicad_sch (KiCad schematic)
At the start: 0 parts

Commit message: Finish input stage schematic
Other:
- sheet dlatch: file 8DLATCH/dlatch/dlatch.kicad_sch -> dlatch/dlatch.kicad_sch
- sheet dlatch1: file 8DLATCH/dlatch/dlatch.kicad_sch -> dlatch/dlatch.kicad_sch
- sheet dlatch2: file 8DLATCH/dlatch/dlatch.kicad_sch -> dlatch/dlatch.kicad_sch
- sheet dlatch3: file 8DLATCH/dlatch/dlatch.kicad_sch -> dlatch/dlatch.kicad_sch
- sheet dlatch4: file 8DLATCH/dlatch/dlatch.kicad_sch -> dlatch/dlatch.kicad_sch
- sheet dlatch5: file 8DLATCH/dlatch/dlatch.kicad_sch -> dlatch/dlatch.kicad_sch
- sheet dlatch6: file 8DLATCH/dlatch/dlatch.kicad_sch -> dlatch/dlatch.kicad_sch
- sheet dlatch7: file 8DLATCH/dlatch/dlatch.kicad_sch -> dlatch/dlatch.kicad_sch
Changed lines of the file:
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@@
 			)
 		)
-		(property "Sheetfile" "8DLATCH/dlatch/dlatch.kicad_sch"
+		(property "Sheetfile" "dlatch/dlatch.kicad_sch"
 			(at 50.8 103.4546 0)
 			(show_name no)
@@
 			)
 		)
-		(property "Sheetfile" "8DLATCH/dlatch/dlatch.kicad_sch"
+		(property "Sheetfile" "dlatch/dlatch.kicad_sch"
 			(at 50.8 126.3146 0)
 			(show_name no)
@@
 			)
 		)
-		(property "Sheetfile" "8DLATCH/dlatch/dlatch.kicad_sch"
+		(property "Sheetfile" "dlatch/dlatch.kicad_sch"
 			(at 50.8 114.8846 0)
 			(show_name no)
@@
 			)
 		)
-		(property "Sheetfile" "8DLATCH/dlatch/dlatch.kicad_sch"
+		(property "Sheetfile" "dlatch/dlatch.kicad_sch"
 			(at 50.8 57.7346 0)
 			(show_name no)
@@
 			)
 		)
-		(property "Sheetfile" "8DLATCH/dlatch/dlatch.kicad_sch"
+		(property "Sheetfile" "dlatch/dlatch.kicad_sch"
 			(at 50.8 69.1646 0)
 			(show_name no)
@@
 			)
 		)
-		(property "Sheetfile" "8DLATCH/dlatch/dlatch.kicad_sch"
+		(property "Sheetfile" "dlatch/dlatch.kicad_sch"
 			(at 50.8 92.0246 0)
 			(show_name no)
@@
 			)
 		)
-		(property "Sheetfile" "8DLATCH/dlatch/dlatch.kicad_sch"
+		(property "Sheetfile" "dlatch/dlatch.kicad_sch"
 			(at 50.8 46.3046 0)
 			(show_name no)
@@
 			)
 		)
-		(property "Sheetfile" "8DLATCH/dlatch/dlatch.kicad_sch"
+		(property "Sheetfile" "dlatch/dlatch.kicad_sch"
 			(at 50.8 80.5946 0)
 			(show_name no)
