File: kicad/controllerBoard/8_1TO2_DEMUX/8_1TO2_DEMUX.kicad_sch (KiCad schematic)
At the start: 0 parts

Commit message: finish address to bit line decoder
Other:
- added sheet 1TO2_DEMUX (1TO2_DEMUX/1TO2_DEMUX.kicad_sch)
- added sheet 1TO2_DEMUX1 (1TO2_DEMUX/1TO2_DEMUX.kicad_sch)
- added sheet 1TO2_DEMUX2 (1TO2_DEMUX/1TO2_DEMUX.kicad_sch)
- added sheet 1TO2_DEMUX3 (1TO2_DEMUX/1TO2_DEMUX.kicad_sch)
- added sheet 1TO2_DEMUX4 (1TO2_DEMUX/1TO2_DEMUX.kicad_sch)
- added sheet 1TO2_DEMUX5 (1TO2_DEMUX/1TO2_DEMUX.kicad_sch)
- added sheet 1TO2_DEMUX6 (1TO2_DEMUX/1TO2_DEMUX.kicad_sch)
- added sheet 1TO2_DEMUX7 (1TO2_DEMUX/1TO2_DEMUX.kicad_sch)
- note added: "Same data, different ADDR to each one. On write, data will be HIGH to pull one of the bit lines LOW. On read, data will be LOW so no bitlines pulled LOW."
