File: kicad/controllerBoard/8_1TO2_DEMUX/1TO2_DEMUX/1TO2_DEMUX.kicad_sch (KiCad schematic)
At the start: 10 parts, among them Q1 PMOS, Q10 NMOS, Q2 NMOS, Q3 PMOS, Q4 PMOS, Q5 PMOS, Q6 NMOS, Q7 NMOS, Q8 PMOS, Q9 NMOS

Commit message: update main board schematic
Parts:
- Q1, Q3, Q4, Q5, Q8: value PMOS -> Q_PMOS_GSD; footprint Package_TO_SOT_SMD:SOT-23-P -> easyeda2kicad:SOT-23-P; symbol Simulation_SPICE:PMOS -> Transistor_FET:Q_PMOS_GSD
- Q10, Q2, Q6, Q7, Q9: value NMOS -> Q_NMOS_GSD; footprint Package_TO_SOT_SMD:SOT-23-N -> easyeda2kicad:SOT-23-N; symbol Simulation_SPICE:NMOS -> Transistor_FET:Q_NMOS_GSD
Connections:
- net +5V: now also Q1.2 (S), Q3.2 (S), Q4.2 (S), Q5.2 (S), Q8.2 (S); no longer Q1.3 (S), Q3.3 (S), Q4.3 (S), Q5.3 (S), Q8.3 (S)
- net Addr: now also Q1.1 (G), Q2.1 (G), Q5.1 (G), Q6.1 (G); no longer Q1.2 (G), Q2.2 (G), Q5.2 (G), Q6.2 (G)
- net D: now also Q10.1 (G), Q3.1 (G), Q4.1 (G), Q7.1 (G); no longer Q10.2 (G), Q3.2 (G), Q4.2 (G), Q7.2 (G)
- net GND: now also Q10.2 (S), Q2.2 (S), Q7.2 (S); no longer Q10.3 (S), Q2.3 (S), Q7.3 (S)
- net ~{Y_{0}}: now also Q4.3 (D), Q8.3 (D), Q9.3 (D); no longer Q4.1 (D), Q8.1 (D), Q9.1 (D)
- net ~{Y_{1}}: now also Q3.3 (D), Q5.3 (D), Q6.3 (D); no longer Q3.1 (D), Q5.1 (D), Q6.1 (D)
- new net: Q1.3 (D), Q2.3 (D), Q8.1 (G), Q9.1 (G)
- new net: Q10.3 (D), Q9.2 (S)
- new net: Q6.2 (S), Q7.3 (D)
Changed lines of the file:
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@@
 	)
 	(symbol
-		(lib_id "Simulation_SPICE:NMOS")
+		(lib_id "Transistor_FET:Q_NMOS_GSD")
 		(at 134.62 111.76 0)
 		(unit 1)
@@
 			)
 		)
-		(property "Value" "NMOS"
+		(property "Value" "Q_NMOS_GSD"
 			(at 140.97 113.0299 0)
 			(show_name no)
@@
 			)
 		)
-		(property "Footprint" "Package_TO_SOT_SMD:SOT-23-N"
+		(property "Footprint" "easyeda2kicad:SOT-23-N"
 			(at 139.7 109.22 0)
 			(hide yes)
@@
 				)
 			)
+			(project "1TO2_DEMUX"
+				(path "/a9fbb7ce-5c19-4e4e-9434-494a3bc76b0f"
+					(reference "Q59")
+					(unit 1)
+				)
+			)
 			(project "8_1TO2_DEMUX"
 				(path "/bb4ef1a0-7d11-42d0-80f2-541f93a64f3e/070613f7-cad7-4c93-89cf-54a08696deb9"
@@
 	)
 	(symbol
-		(lib_id "Simulation_SPICE:PMOS")
+		(lib_id "Transistor_FET:Q_PMOS_GSD")
 		(at 118.11 97.79 0)
 		(mirror x)
@@
 			)
 		)
-		(property "Value" "PMOS"
+		(property "Value" "Q_PMOS_GSD"
 			(at 124.46 99.0599 0)
 			(show_name no)
@@
 			)
 		)
-		(property "Footprint" "Package_TO_SOT_SMD:SOT-23-P"
+		(property "Footprint" "easyeda2kicad:SOT-23-P"
 			(at 123.19 100.33 0)
 			(hide yes)
@@
 				)
 			)
+			(project "1TO2_DEMUX"
+				(path "/a9fbb7ce-5c19-4e4e-9434-494a3bc76b0f"
+					(reference "Q54")
+					(unit 1)
+				)
+			)
 			(project "8_1TO2_DEMUX"
 				(path "/bb4ef1a0-7d11-42d0-80f2-541f93a64f3e/070613f7-cad7-4c93-89cf-54a08696deb9"
@@
 	)
 	(symbol
-		(lib_id "Simulation_SPICE:PMOS")
+		(lib_id "Transistor_FET:Q_PMOS_GSD")
 		(at 121.92 31.75 0)
 		(mirror x)
@@
 			)
 		)
-		(property "Value" "PMOS"
+		(property "Value" "Q_PMOS_GSD"
 			(at 128.27 33.0199 0)
 			(show_name no)
@@
 			)
 		)
-		(property "Footprint" "Package_TO_SOT_SMD:SOT-23-P"
+		(property "Footprint" "easyeda2kicad:SOT-23-P"
 			(at 127 34.29 0)
 			(hide yes)
@@
 				(path "/93a9a1ca-4ee5-40da-ab67-92836146c003/8a491917-4253-4ca5-a31e-fc7dcc04a377/e3920536-71f2-4b6c-a5bc-cfcc9ab0bde8"
 					(reference "Q35")
+					(unit 1)
+				)
+			)
+			(project "1TO2_DEMUX"
+				(path "/a9fbb7ce-5c19-4e4e-9434-494a3bc76b0f"
+					(reference "Q55")
 					(unit 1)
 				)
@@
 				)
 			)
+			(project "1TO2_DEMUX"
+				(path "/a9fbb7ce-5c19-4e4e-9434-494a3bc76b0f"
+					(reference "#PWR037")
+					(unit 1)
+				)
+			)
 			(project "8_1TO2_DEMUX"
 				(path "/bb4ef1a0-7d11-42d0-80f2-541f93a64f3e/070613f7-cad7-4c93-89cf-54a08696deb9"
@@
 				)
 			)
+			(project "1TO2_DEMUX"
+				(path "/a9fbb7ce-5c19-4e4e-9434-494a3bc76b0f"
+					(reference "#PWR042")
+					(unit 1)
+				)
+			)
 			(project "8_1TO2_DEMUX"
 				(path "/bb4ef1a0-7d11-42d0-80f2-541f93a64f3e/070613f7-cad7-4c93-89cf-54a08696deb9"
@@
 				)
 			)
+			(project "1TO2_DEMUX"
+				(path "/a9fbb7ce-5c19-4e4e-9434-494a3bc76b0f"
+					(reference "#PWR040")
+					(unit 1)
+				)
+			)
 			(project "8_1TO2_DEMUX"
 				(path "/bb4ef1a0-7d11-42d0-80f2-541f93a64f3e/070613f7-cad7-4c93-89cf-54a08696deb9"
@@
 	)
 	(symbol
-		(lib_id "Simulation_SPICE:NMOS")
+		(lib_id "Transistor_FET:Q_NMOS_GSD")
 		(at 121.92 45.72 0)
 		(unit 1)
@@
 			)
 		)
-		(property "Value" "NMOS"
+		(property "Value" "Q_NMOS_GSD"
 			(at 128.27 46.9899 0)
 			(show_name no)
@@
 			)
 		)
-		(property "Footprint" "Package_TO_SOT_SMD:SOT-23-N"
+		(property "Footprint" "easyeda2kicad:SOT-23-N"
 			(at 127 43.18 0)
 			(hide yes)
@@
 				)
 			)
+			(project "1TO2_DEMUX"
+				(path "/a9fbb7ce-5c19-4e4e-9434-494a3bc76b0f"
+					(reference "Q56")
+					(unit 1)
+				)
+			)
 			(project "8_1TO2_DEMUX"
 				(path "/bb4ef1a0-7d11-42d0-80f2-541f93a64f3e/070613f7-cad7-4c93-89cf-54a08696deb9"
@@
 	)
 	(symbol
-		(lib_id "Simulation_SPICE:PMOS")
+		(lib_id "Transistor_FET:Q_PMOS_GSD")
 		(at 134.62 97.79 0)
 		(mirror x)
@@
 			)
 		)
-		(property "Value" "PMOS"
+		(property "Value" "Q_PMOS_GSD"
 			(at 140.97 99.0599 0)
 			(show_name no)
@@
 			)
 		)
-		(property "Footprint" "Package_TO_SOT_SMD:SOT-23-P"
+		(property "Footprint" "easyeda2kicad:SOT-23-P"
 			(at 139.7 100.33 0)
 			(hide yes)
@@
 				)
 			)
+			(project "1TO2_DEMUX"
+				(path "/a9fbb7ce-5c19-4e4e-9434-494a3bc76b0f"
+					(reference "Q58")
+					(unit 1)
+				)
+			)
 			(project "8_1TO2_DEMUX"
 				(path "/bb4ef1a0-7d11-42d0-80f2-541f93a64f3e/070613f7-cad7-4c93-89cf-54a08696deb9"
@@
 	)
 	(symbol
-		(lib_id "Simulation_SPICE:NMOS")
+		(lib_id "Transistor_FET:Q_NMOS_GSD")
 		(at 121.92 55.88 0)
 		(unit 1)
@@
 			)
 		)
-		(property "Value" "NMOS"
+		(property "Value" "Q_NMOS_GSD"
 			(at 128.27 57.1499 0)
 			(show_name no)
@@
 			)
 		)
-		(property "Footprint" "Package_TO_SOT_SMD:SOT-23-N"
+		(property "Footprint" "easyeda2kicad:SOT-23-N"
 			(at 127 53.34 0)
 			(hide yes)
@@
 				)
 			)
+			(project "1TO2_DEMUX"
+				(path "/a9fbb7ce-5c19-4e4e-9434-494a3bc76b0f"
+					(reference "Q57")
+					(unit 1)
+				)
+			)
 			(project "8_1TO2_DEMUX"
 				(path "/bb4ef1a0-7d11-42d0-80f2-541f93a64f3e/070613f7-cad7-4c93-89cf-54a08696deb9"
@@
 	)
 	(symbol
-		(lib_id "Simulation_SPICE:PMOS")
+		(lib_id "Transistor_FET:Q_PMOS_GSD")
 		(at 105.41 31.75 0)
 		(mirror x)
@@
 			)
 		)
-		(property "Value" "PMOS"
+		(property "Value" "Q_PMOS_GSD"
 			(at 111.76 33.0199 0)
 			(show_name no)
@@
 			)
 		)
-		(property "Footprint" "Package_TO_SOT_SMD:SOT-23-P"
+		(property "Footprint" "easyeda2kicad:SOT-23-P"
 			(at 110.49 34.29 0)
 			(hide yes)
@@
 				(path "/93a9a1ca-4ee5-40da-ab67-92836146c003/8a491917-4253-4ca5-a31e-fc7dcc04a377/e3920536-71f2-4b6c-a5bc-cfcc9ab0bde8"
 					(reference "Q33")
+					(unit 1)
+				)
+			)
+			(project "1TO2_DEMUX"
+				(path "/a9fbb7ce-5c19-4e4e-9434-494a3bc76b0f"
+					(reference "Q53")
 					(unit 1)
 				)
@@
 				)
 			)
+			(project "1TO2_DEMUX"
+				(path "/a9fbb7ce-5c19-4e4e-9434-494a3bc76b0f"
+					(reference "#PWR041")
+					(unit 1)
+				)
+			)
 			(project "8_1TO2_DEMUX"
 				(path "/bb4ef1a0-7d11-42d0-80f2-541f93a64f3e/070613f7-cad7-4c93-89cf-54a08696deb9"
@@
 	)
 	(symbol
-		(lib_id "Simulation_SPICE:NMOS")
+		(lib_id "Transistor_FET:Q_NMOS_GSD")
 		(at 80.01 95.25 0)
 		(unit 1)
@@
 			)
 		)
-		(property "Value" "NMOS"
+		(property "Value" "Q_NMOS_GSD"
 			(at 86.36 96.5199 0)
 			(show_name no)
@@
 			)
 		)
-		(property "Footprint" "Package_TO_SOT_SMD:SOT-23-N"
+		(property "Footprint" "easyeda2kicad:SOT-23-N"
 			(at 85.09 92.71 0)
 			(hide yes)
@@
 				)
 			)
+			(project "1TO2_DEMUX"
+				(path "/a9fbb7ce-5c19-4e4e-9434-494a3bc76b0f"
+					(reference "Q52")
+					(unit 1)
+				)
+			)
 			(project "8_1TO2_DEMUX"
 				(path "/bb4ef1a0-7d11-42d0-80f2-541f93a64f3e/070613f7-cad7-4c93-89cf-54a08696deb9"
@@
 	)
 	(symbol
-		(lib_id "Simulation_SPICE:NMOS")
+		(lib_id "Transistor_FET:Q_NMOS_GSD")
 		(at 134.62 121.92 0)
 		(unit 1)
@@
 			)
 		)
-		(property "Value" "NMOS"
+		(property "Value" "Q_NMOS_GSD"
 			(at 140.97 123.1899 0)
 			(show_name no)
@@
 			)
 		)
-		(property "Footprint" "Package_TO_SOT_SMD:SOT-23-N"
+		(property "Footprint" "easyeda2kicad:SOT-23-N"
 			(at 139.7 119.38 0)
 			(hide yes)
@@
 				(path "/93a9a1ca-4ee5-40da-ab67-92836146c003/8a491917-4253-4ca5-a31e-fc7dcc04a377/e3920536-71f2-4b6c-a5bc-cfcc9ab0bde8"
 					(reference "Q40")
+					(unit 1)
+				)
+			)
+			(project "1TO2_DEMUX"
+				(path "/a9fbb7ce-5c19-4e4e-9434-494a3bc76b0f"
+					(reference "Q60")
 					(unit 1)
 				)
@@
 				)
 			)
+			(project "1TO2_DEMUX"
+				(path "/a9fbb7ce-5c19-4e4e-9434-494a3bc76b0f"
+					(reference "#PWR039")
+					(unit 1)
+				)
+			)
 			(project "8_1TO2_DEMUX"
 				(path "/bb4ef1a0-7d11-42d0-80f2-541f93a64f3e/070613f7-cad7-4c93-89cf-54a08696deb9"
@@
 	)
 	(symbol
-		(lib_id "Simulation_SPICE:PMOS")
+		(lib_id "Transistor_FET:Q_PMOS_GSD")
 		(at 80.01 85.09 0)
 		(mirror x)
@@
 			)
 		)
-		(property "Value" "PMOS"
+		(property "Value" "Q_PMOS_GSD"
 			(at 86.36 86.3599 0)
 			(show_name no)
@@
 			)
 		)
-		(property "Footprint" "Package_TO_SOT_SMD:SOT-23-P"
+		(property "Footprint" "easyeda2kicad:SOT-23-P"
 			(at 85.09 87.63 0)
 			(hide yes)
@@
 				(path "/93a9a1ca-4ee5-40da-ab67-92836146c003/8a491917-4253-4ca5-a31e-fc7dcc04a377/e3920536-71f2-4b6c-a5bc-cfcc9ab0bde8"
 					(reference "Q31")
+					(unit 1)
+				)
+			)
+			(project "1TO2_DEMUX"
+				(path "/a9fbb7ce-5c19-4e4e-9434-494a3bc76b0f"
+					(reference "Q51")
 					(unit 1)
 				)
@@
 				)
 			)
+			(project "1TO2_DEMUX"
+				(path "/a9fbb7ce-5c19-4e4e-9434-494a3bc76b0f"
+					(reference "#PWR038")
+					(unit 1)
+				)
+			)
 			(project "8_1TO2_DEMUX"
 				(path "/bb4ef1a0-7d11-42d0-80f2-541f93a64f3e/070613f7-cad7-4c93-89cf-54a08696deb9"
@@
 		)
 	)
+	(sheet_instances
+		(path "/"
+			(page "1")
+		)
+	)
