File: kicad/controllerBoard/5V_TO_10V/5V_TO_10V.kicad_pcb (KiCad board)
At the start: 2 copper layers, 51 parts, among them Q1 Q_PMOS_GSD, Q10 Q_NMOS_GSD, Q11 Q_PMOS_GSD, Q12 Q_NMOS_GSD, Q13 Q_PMOS_GSD, Q14 Q_NMOS_GSD, Q15 Q_PMOS_GSD, Q16 Q_NMOS_GSD, Q17 Q_PMOS_GSD, Q18 Q_NMOS_GSD, Q2 Q_PMOS_GSD, Q3 Q_NMOS_GSD, Q4 Q_NMOS_GSD, Q5 Q_PMOS_GSD, Q6 Q_NMOS_GSD, Q7 Q_PMOS_GSD, Q8 Q_NMOS_GSD, Q9 Q_PMOS_GSD

Commit message: add mounting holes
Parts:
- moved D1 6.00 mm to (102.0, 73.0)
- moved C8 1.20 mm to (100.5, 64.0), turned to 0 degrees
Routing:
- net +5V: track 37.2 -> 42.6 mm, vias 18 -> 24
- net Net-(D1-K): track 16.8 -> 19.3 mm
- net GND: track 33.7 -> 33.2 mm
