File: kicad/controllerBoard/RISING_EDGE_DETECTOR/RISING_EDGE_DETECTOR.kicad_pcb (KiCad board)
At the start: 2 copper layers, 29 parts, among them Q1 Q_PMOS_GSD, Q10 Q_PMOS_GSD, Q11 Q_NMOS_GSD, Q12 Q_NMOS_GSD, Q13 Q_PMOS_GSD, Q14 Q_NMOS_GSD, Q2 Q_NMOS_GSD, Q3 Q_PMOS_GSD, Q4 Q_NMOS_GSD, Q5 Q_PMOS_GSD, Q6 Q_NMOS_GSD, Q7 Q_PMOS_GSD, Q8 Q_NMOS_GSD, Q9 Q_PMOS_GSD

Commit message: Add breakout board through holes on main ram board
Routing:
- net GND: track 14.8 -> 16.9 mm, vias 6 -> 7
