File: kicad/controllerBoard/WL_PULSE_GEN/WL_PULSE_GEN.kicad_pcb (KiCad board)
At the start: 2 copper layers, 20 parts, among them Q1 Q_PMOS_GSD, Q2 Q_NMOS_GSD, Q3 Q_PMOS_GSD, Q4 Q_NMOS_GSD, Q5 Q_PMOS_GSD, Q6 Q_NMOS_GSD, Q7 Q_PMOS_GSD, Q8 Q_NMOS_GSD

Commit message: Add breakout board through holes on main ram board
Routing:
- net +5V: track 9.11 -> 10.6 mm, vias 5 -> 6
