File: kicad/controllerBoard/WL_PULSE_GEN/WL_PULSE_GEN.kicad_sch (KiCad schematic)
At the start: 18 parts, among them Q409 PMOS, Q410 NMOS, Q411 PMOS, Q412 NMOS, Q413 PMOS, Q414 NMOS, Q415 PMOS, Q416 NMOS

Commit message: did stuff
Parts:
- renumbered C4 to C10, C2 to C8, C3 to C9, D2 to D4, Q409 to Q412, Q410 to Q413, Q411 to Q414, Q412 to Q415, Q413 to Q416, Q414 to Q417, Q415 to Q418, Q416 to Q419, R27 to R34, R28 to R35, R29 to R36, R30 to R37, R31 to R38, R32 to R39
Changed lines of the file:
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@@
 		(dnp no)
 		(fields_autoplaced yes)
-		(property "Reference" "#PWR03"
+		(property "Reference" "#PWR0102"
 			(at 113.03 100.33 0)
 			(hide yes)
@@
 			(project "controllerBoard"
 				(path "/93a9a1ca-4ee5-40da-ab67-92836146c003/8b3cd8c5-d66b-460c-b4ee-229e25c1238a"
-					(reference "#PWR03")
+					(reference "#PWR0102")
 					(unit 1)
 				)
@@
 		(dnp no)
 		(fields_autoplaced yes)
-		(property "Reference" "R27"
+		(property "Reference" "R34"
 			(at 91.44 78.7399 0)
 			(show_name no)
@@
 			(project "controllerBoard"
 				(path "/93a9a1ca-4ee5-40da-ab67-92836146c003/8b3cd8c5-d66b-460c-b4ee-229e25c1238a"
-					(reference "R27")
+					(reference "R34")
 					(unit 1)
 				)
@@
 		(dnp no)
 		(fields_autoplaced yes)
-		(property "Reference" "Q414"
+		(property "Reference" "Q417"
 			(at 166.37 87.6299 0)
 			(show_name no)
@@
 			(project "controllerBoard"
 				(path "/93a9a1ca-4ee5-40da-ab67-92836146c003/8b3cd8c5-d66b-460c-b4ee-229e25c1238a"
-					(reference "Q414")
+					(reference "Q417")
 					(unit 1)
 				)
@@
 		(dnp no)
 		(fields_autoplaced yes)
-		(property "Reference" "Q411"
+		(property "Reference" "Q414"
 			(at 142.24 62.2299 0)
 			(show_name no)
@@
 			(project "controllerBoard"
 				(path "/93a9a1ca-4ee5-40da-ab67-92836146c003/8b3cd8c5-d66b-460c-b4ee-229e25c1238a"
-					(reference "Q411")
+					(reference "Q414")
 					(unit 1)
 				)
@@
 		(dnp no)
 		(fields_autoplaced yes)
-		(property "Reference" "D2"
+		(property "Reference" "D4"
 			(at 101.6 78.7399 90)
 			(show_name no)
@@
 			(project "controllerBoard"
 				(path "/93a9a1ca-4ee5-40da-ab67-92836146c003/8b3cd8c5-d66b-460c-b4ee-229e25c1238a"
-					(reference "D2")
+					(reference "D4")
 					(unit 1)
 				)
@@
 		(dnp no)
 		(fields_autoplaced yes)
-		(property "Reference" "Q415"
+		(property "Reference" "Q418"
 			(at 191.77 62.2299 0)
 			(show_name no)
@@
 			(project "controllerBoard"
 				(path "/93a9a1ca-4ee5-40da-ab67-92836146c003/8b3cd8c5-d66b-460c-b4ee-229e25c1238a"
-					(reference "Q415")
+					(reference "Q418")
 					(unit 1)
 				)
@@
 		(dnp no)
 		(fields_autoplaced yes)
-		(property "Reference" "Q410"
+		(property "Reference" "Q413"
 			(at 116.84 87.6299 0)
 			(show_name no)
@@
 			(project "controllerBoard"
 				(path "/93a9a1ca-4ee5-40da-ab67-92836146c003/8b3cd8c5-d66b-460c-b4ee-229e25c1238a"
-					(reference "Q410")
+					(reference "Q413")
 					(unit 1)
 				)
@@
 		(dnp no)
 		(fields_autoplaced yes)
-		(property "Reference" "Q413"
+		(property "Reference" "Q416"
 			(at 166.37 62.2299 0)
 			(show_name no)
@@
 			(project "controllerBoard"
 				(path "/93a9a1ca-4ee5-40da-ab67-92836146c003/8b3cd8c5-d66b-460c-b4ee-229e25c1238a"
-					(reference "Q413")
+					(reference "Q416")
 					(unit 1)
 				)
@@
 		(dnp no)
 		(fields_autoplaced yes)
-		(property "Reference" "C2"
+		(property "Reference" "C8"
 			(at 85.09 68.58 90)
 			(show_name no)
@@
 			(project "controllerBoard"
 				(path "/93a9a1ca-4ee5-40da-ab67-92836146c003/8b3cd8c5-d66b-460c-b4ee-229e25c1238a"
-					(reference "C2")
+					(reference "C8")
 					(unit 1)
 				)
@@
 		(dnp no)
 		(fields_autoplaced yes)
-		(property "Reference" "#PWR05"
+		(property "Reference" "#PWR0103"
 			(at 123.19 90.17 0)
 			(hide yes)
@@
 			(project "controllerBoard"
 				(path "/93a9a1ca-4ee5-40da-ab67-92836146c003/8b3cd8c5-d66b-460c-b4ee-229e25c1238a"
-					(reference "#PWR05")
+					(reference "#PWR0103")
 					(unit 1)
 				)
@@
 		(dnp no)
 		(fields_autoplaced yes)
-		(property "Reference" "#PWR02"
+		(property "Reference" "#PWR0101"
 			(at 99.06 90.17 0)
 			(hide yes)
@@
 			(project "controllerBoard"
 				(path "/93a9a1ca-4ee5-40da-ab67-92836146c003/8b3cd8c5-d66b-460c-b4ee-229e25c1238a"
-					(reference "#PWR02")
+					(reference "#PWR0101")
 					(unit 1)
 				)
@@
 		(dnp no)
 		(fields_autoplaced yes)
-		(property "Reference" "R29"
+		(property "Reference" "R36"
 			(at 115.57 78.7399 0)
 			(show_name no)
@@
 			(project "controllerBoard"
 				(path "/93a9a1ca-4ee5-40da-ab67-92836146c003/8b3cd8c5-d66b-460c-b4ee-229e25c1238a"
-					(reference "R29")
+					(reference "R36")
 					(unit 1)
 				)
@@
 		(dnp no)
 		(fields_autoplaced yes)
-		(property "Reference" "#PWR09"
+		(property "Reference" "#PWR0106"
 			(at 148.59 62.23 0)
 			(hide yes)
@@
 			(project "controllerBoard"
 				(path "/93a9a1ca-4ee5-40da-ab67-92836146c003/8b3cd8c5-d66b-460c-b4ee-229e25c1238a"
-					(reference "#PWR09")
+					(reference "#PWR0106")
 					(unit 1)
 				)
@@
 		(dnp no)
 		(fields_autoplaced yes)
-		(property "Reference" "#PWR08"
+		(property "Reference" "#PWR0105"
 			(at 147.32 90.17 0)
 			(hide yes)
@@
 			(project "controllerBoard"
 				(path "/93a9a1ca-4ee5-40da-ab67-92836146c003/8b3cd8c5-d66b-460c-b4ee-229e25c1238a"
-					(reference "#PWR08")
+					(reference "#PWR0105")
 					(unit 1)
 				)
@@
 		(dnp no)
 		(fields_autoplaced yes)
-		(property "Reference" "C3"
+		(property "Reference" "C9"
 			(at 127 78.7399 0)
 			(show_name no)
@@
 			(project "controllerBoard"
 				(path "/93a9a1ca-4ee5-40da-ab67-92836146c003/8b3cd8c5-d66b-460c-b4ee-229e25c1238a"
-					(reference "C3")
+					(reference "C9")
 					(unit 1)
 				)
@@
 		(dnp no)
 		(fields_autoplaced yes)
-		(property "Reference" "C4"
+		(property "Reference" "C10"
 			(at 151.13 78.7399 0)
 			(show_name no)
@@
 			(project "controllerBoard"
 				(path "/93a9a1ca-4ee5-40da-ab67-92836146c003/8b3cd8c5-d66b-460c-b4ee-229e25c1238a"
-					(reference "C4")
+					(reference "C10")
 					(unit 1)
 				)
@@
 		(dnp no)
 		(fields_autoplaced yes)
-		(property "Reference" "Q416"
+		(property "Reference" "Q419"
 			(at 191.77 87.6299 0)
 			(show_name no)
@@
 			(project "controllerBoard"
 				(path "/93a9a1ca-4ee5-40da-ab67-92836146c003/8b3cd8c5-d66b-460c-b4ee-229e25c1238a"
-					(reference "Q416")
+					(reference "Q419")
 					(unit 1)
 				)
@@
 		(dnp no)
 		(fields_autoplaced yes)
-		(property "Reference" "Q412"
+		(property "Reference" "Q415"
 			(at 142.24 87.6299 0)
 			(show_name no)
@@
 			(project "controllerBoard"
 				(path "/93a9a1ca-4ee5-40da-ab67-92836146c003/8b3cd8c5-d66b-460c-b4ee-229e25c1238a"
-					(reference "Q412")
+					(reference "Q415")
 					(unit 1)
 				)
@@
 		(dnp no)
 		(fields_autoplaced yes)
-		(property "Reference" "R30"
+		(property "Reference" "R37"
 			(at 140.97 71.1199 0)
 			(show_name no)
@@
 			(project "controllerBoard"
 				(path "/93a9a1ca-4ee5-40da-ab67-92836146c003/8b3cd8c5-d66b-460c-b4ee-229e25c1238a"
-					(reference "R30")
+					(reference "R37")
 					(unit 1)
 				)
@@
 		(dnp no)
 		(fields_autoplaced yes)
-		(property "Reference" "R28"
+		(property "Reference" "R35"
 			(at 115.57 71.1199 0)
 			(show_name no)
@@
 			(project "controllerBoard"
 				(path "/93a9a1ca-4ee5-40da-ab67-92836146c003/8b3cd8c5-d66b-460c-b4ee-229e25c1238a"
-					(reference "R28")
+					(reference "R35")
 					(unit 1)
 				)
@@
 		(dnp no)
 		(fields_autoplaced yes)
-		(property "Reference" "#PWR01"
+		(property "Reference" "#PWR0100"
 			(at 88.9 90.17 0)
 			(hide yes)
@@
 			(project "controllerBoard"
 				(path "/93a9a1ca-4ee5-40da-ab67-92836146c003/8b3cd8c5-d66b-460c-b4ee-229e25c1238a"
-					(reference "#PWR01")
+					(reference "#PWR0100")
 					(unit 1)
 				)
@@
 		(dnp no)
 		(fields_autoplaced yes)
-		(property "Reference" "#PWR07"
+		(property "Reference" "#PWR0108"
 			(at 187.96 100.33 0)
 			(hide yes)
@@
 			(project "controllerBoard"
 				(path "/93a9a1ca-4ee5-40da-ab67-92836146c003/8b3cd8c5-d66b-460c-b4ee-229e25c1238a"
-					(reference "#PWR07")
+					(reference "#PWR0108")
 					(unit 1)
 				)
@@
 		(dnp no)
 		(fields_autoplaced yes)
-		(property "Reference" "#PWR04"
+		(property "Reference" "#PWR0104"
 			(at 138.43 100.33 0)
 			(hide yes)
@@
 			(project "controllerBoard"
 				(path "/93a9a1ca-4ee5-40da-ab67-92836146c003/8b3cd8c5-d66b-460c-b4ee-229e25c1238a"
-					(reference "#PWR04")
+					(reference "#PWR0104")
 					(unit 1)
 				)
@@
 		(dnp no)
 		(fields_autoplaced yes)
-		(property "Reference" "R31"
+		(property "Reference" "R38"
 			(at 165.1 71.1199 0)
 			(show_name no)
@@
 			(project "controllerBoard"
 				(path "/93a9a1ca-4ee5-40da-ab67-92836146c003/8b3cd8c5-d66b-460c-b4ee-229e25c1238a"
-					(reference "R31")
+					(reference "R38")
 					(unit 1)
 				)
@@
 		(dnp no)
 		(fields_autoplaced yes)
-		(property "Reference" "Q409"
+		(property "Reference" "Q412"
 			(at 116.84 62.2299 0)
 			(show_name no)
@@
 			(project "controllerBoard"
 				(path "/93a9a1ca-4ee5-40da-ab67-92836146c003/8b3cd8c5-d66b-460c-b4ee-229e25c1238a"
-					(reference "Q409")
+					(reference "Q412")
 					(unit 1)
 				)
@@
 		(dnp no)
 		(fields_autoplaced yes)
-		(property "Reference" "R32"
+		(property "Reference" "R39"
 			(at 190.5 71.1199 0)
 			(show_name no)
@@
 			(project "controllerBoard"
 				(path "/93a9a1ca-4ee5-40da-ab67-92836146c003/8b3cd8c5-d66b-460c-b4ee-229e25c1238a"
-					(reference "R32")
+					(reference "R39")
 					(unit 1)
 				)
@@
 		(dnp no)
 		(fields_autoplaced yes)
-		(property "Reference" "#PWR06"
+		(property "Reference" "#PWR0107"
 			(at 162.56 100.33 0)
 			(hide yes)
@@
 			(project "controllerBoard"
 				(path "/93a9a1ca-4ee5-40da-ab67-92836146c003/8b3cd8c5-d66b-460c-b4ee-229e25c1238a"
-					(reference "#PWR06")
-					(unit 1)
-				)
+					(reference "#PWR0107")
+					(unit 1)
+				)

Commit message: did more simulation, added bom
Parts:
- renumbered C8 to C4, C9 to C5, C10 to C6, D4 to D2, Q412 to Q405, Q413 to Q406, Q414 to Q407, Q415 to Q408, Q416 to Q409, Q417 to Q410, Q418 to Q411, Q419 to Q412, R34 to R22, R35 to R23, R36 to R24, R37 to R25, R38 to R26, R39 to R27
Changed lines of the file:
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@@
 		(dnp no)
 		(fields_autoplaced yes)
-		(property "Reference" "#PWR0102"
+		(property "Reference" "#PWR096"
 			(at 113.03 100.33 0)
 			(hide yes)
@@
 			(project "controllerBoard"
 				(path "/93a9a1ca-4ee5-40da-ab67-92836146c003/8b3cd8c5-d66b-460c-b4ee-229e25c1238a"
-					(reference "#PWR0102")
+					(reference "#PWR096")
 					(unit 1)
 				)
@@
 		(dnp no)
 		(fields_autoplaced yes)
-		(property "Reference" "R34"
+		(property "Reference" "R22"
 			(at 91.44 78.7399 0)
 			(show_name no)
@@
 			(project "controllerBoard"
 				(path "/93a9a1ca-4ee5-40da-ab67-92836146c003/8b3cd8c5-d66b-460c-b4ee-229e25c1238a"
-					(reference "R34")
+					(reference "R22")
 					(unit 1)
 				)
@@
 		(dnp no)
 		(fields_autoplaced yes)
-		(property "Reference" "Q417"
+		(property "Reference" "Q410"
 			(at 166.37 87.6299 0)
 			(show_name no)
@@
 			(project "controllerBoard"
 				(path "/93a9a1ca-4ee5-40da-ab67-92836146c003/8b3cd8c5-d66b-460c-b4ee-229e25c1238a"
-					(reference "Q417")
+					(reference "Q410")
 					(unit 1)
 				)
@@
 		(dnp no)
 		(fields_autoplaced yes)
-		(property "Reference" "Q414"
+		(property "Reference" "Q407"
 			(at 142.24 62.2299 0)
 			(show_name no)
@@
 			(project "controllerBoard"
 				(path "/93a9a1ca-4ee5-40da-ab67-92836146c003/8b3cd8c5-d66b-460c-b4ee-229e25c1238a"
-					(reference "Q414")
+					(reference "Q407")
 					(unit 1)
 				)
@@
 		(dnp no)
 		(fields_autoplaced yes)
-		(property "Reference" "D4"
+		(property "Reference" "D2"
 			(at 101.6 78.7399 90)
 			(show_name no)
@@
 			(project "controllerBoard"
 				(path "/93a9a1ca-4ee5-40da-ab67-92836146c003/8b3cd8c5-d66b-460c-b4ee-229e25c1238a"
-					(reference "D4")
+					(reference "D2")
 					(unit 1)
 				)
@@
 		(dnp no)
 		(fields_autoplaced yes)
-		(property "Reference" "Q418"
+		(property "Reference" "Q411"
 			(at 191.77 62.2299 0)
 			(show_name no)
@@
 			(project "controllerBoard"
 				(path "/93a9a1ca-4ee5-40da-ab67-92836146c003/8b3cd8c5-d66b-460c-b4ee-229e25c1238a"
-					(reference "Q418")
+					(reference "Q411")
 					(unit 1)
 				)
@@
 		(dnp no)
 		(fields_autoplaced yes)
-		(property "Reference" "Q413"
+		(property "Reference" "Q406"
 			(at 116.84 87.6299 0)
 			(show_name no)
@@
 			(project "controllerBoard"
 				(path "/93a9a1ca-4ee5-40da-ab67-92836146c003/8b3cd8c5-d66b-460c-b4ee-229e25c1238a"
-					(reference "Q413")
+					(reference "Q406")
 					(unit 1)
 				)
@@
 		(dnp no)
 		(fields_autoplaced yes)
-		(property "Reference" "Q416"
+		(property "Reference" "Q409"
 			(at 166.37 62.2299 0)
 			(show_name no)
@@
 			(project "controllerBoard"
 				(path "/93a9a1ca-4ee5-40da-ab67-92836146c003/8b3cd8c5-d66b-460c-b4ee-229e25c1238a"
-					(reference "Q416")
+					(reference "Q409")
 					(unit 1)
 				)
@@
 		(dnp no)
 		(fields_autoplaced yes)
-		(property "Reference" "C8"
+		(property "Reference" "C4"
 			(at 85.09 68.58 90)
 			(show_name no)
@@
 			(project "controllerBoard"
 				(path "/93a9a1ca-4ee5-40da-ab67-92836146c003/8b3cd8c5-d66b-460c-b4ee-229e25c1238a"
-					(reference "C8")
+					(reference "C4")
 					(unit 1)
 				)
@@
 		(dnp no)
 		(fields_autoplaced yes)
-		(property "Reference" "#PWR0103"
+		(property "Reference" "#PWR097"
 			(at 123.19 90.17 0)
 			(hide yes)
@@
 			(project "controllerBoard"
 				(path "/93a9a1ca-4ee5-40da-ab67-92836146c003/8b3cd8c5-d66b-460c-b4ee-229e25c1238a"
-					(reference "#PWR0103")
+					(reference "#PWR097")
 					(unit 1)
 				)
@@
 		(dnp no)
 		(fields_autoplaced yes)
-		(property "Reference" "#PWR0101"
+		(property "Reference" "#PWR095"
 			(at 99.06 90.17 0)
 			(hide yes)
@@
 			(project "controllerBoard"
 				(path "/93a9a1ca-4ee5-40da-ab67-92836146c003/8b3cd8c5-d66b-460c-b4ee-229e25c1238a"
-					(reference "#PWR0101")
+					(reference "#PWR095")
 					(unit 1)
 				)
@@
 		(dnp no)
 		(fields_autoplaced yes)
-		(property "Reference" "R36"
+		(property "Reference" "R24"
 			(at 115.57 78.7399 0)
 			(show_name no)
@@
 			(project "controllerBoard"
 				(path "/93a9a1ca-4ee5-40da-ab67-92836146c003/8b3cd8c5-d66b-460c-b4ee-229e25c1238a"
-					(reference "R36")
+					(reference "R24")
 					(unit 1)
 				)
@@
 		(dnp no)
 		(fields_autoplaced yes)
-		(property "Reference" "#PWR0106"
+		(property "Reference" "#PWR0100"
 			(at 148.59 62.23 0)
 			(hide yes)
@@
 			(project "controllerBoard"
 				(path "/93a9a1ca-4ee5-40da-ab67-92836146c003/8b3cd8c5-d66b-460c-b4ee-229e25c1238a"
-					(reference "#PWR0106")
+					(reference "#PWR0100")
 					(unit 1)
 				)
@@
 		(dnp no)
 		(fields_autoplaced yes)
-		(property "Reference" "#PWR0105"
+		(property "Reference" "#PWR099"
 			(at 147.32 90.17 0)
 			(hide yes)
@@
 			(project "controllerBoard"
 				(path "/93a9a1ca-4ee5-40da-ab67-92836146c003/8b3cd8c5-d66b-460c-b4ee-229e25c1238a"
-					(reference "#PWR0105")
+					(reference "#PWR099")
 					(unit 1)
 				)
@@
 		(dnp no)
 		(fields_autoplaced yes)
-		(property "Reference" "C9"
+		(property "Reference" "C5"
 			(at 127 78.7399 0)
 			(show_name no)
@@
 			(project "controllerBoard"
 				(path "/93a9a1ca-4ee5-40da-ab67-92836146c003/8b3cd8c5-d66b-460c-b4ee-229e25c1238a"
-					(reference "C9")
+					(reference "C5")
 					(unit 1)
 				)
@@
 		(dnp no)
 		(fields_autoplaced yes)
-		(property "Reference" "C10"
+		(property "Reference" "C6"
 			(at 151.13 78.7399 0)
 			(show_name no)
@@
 			(project "controllerBoard"
 				(path "/93a9a1ca-4ee5-40da-ab67-92836146c003/8b3cd8c5-d66b-460c-b4ee-229e25c1238a"
-					(reference "C10")
+					(reference "C6")
 					(unit 1)
 				)
@@
 		(dnp no)
 		(fields_autoplaced yes)
-		(property "Reference" "Q419"
+		(property "Reference" "Q412"
 			(at 191.77 87.6299 0)
 			(show_name no)
@@
 			(project "controllerBoard"
 				(path "/93a9a1ca-4ee5-40da-ab67-92836146c003/8b3cd8c5-d66b-460c-b4ee-229e25c1238a"
-					(reference "Q419")
+					(reference "Q412")
 					(unit 1)
 				)
@@
 		(dnp no)
 		(fields_autoplaced yes)
-		(property "Reference" "Q415"
+		(property "Reference" "Q408"
 			(at 142.24 87.6299 0)
 			(show_name no)
@@
 			(project "controllerBoard"
 				(path "/93a9a1ca-4ee5-40da-ab67-92836146c003/8b3cd8c5-d66b-460c-b4ee-229e25c1238a"
-					(reference "Q415")
+					(reference "Q408")
 					(unit 1)
 				)
@@
 		(dnp no)
 		(fields_autoplaced yes)
-		(property "Reference" "R37"
+		(property "Reference" "R25"
 			(at 140.97 71.1199 0)
 			(show_name no)
@@
 			(project "controllerBoard"
 				(path "/93a9a1ca-4ee5-40da-ab67-92836146c003/8b3cd8c5-d66b-460c-b4ee-229e25c1238a"
-					(reference "R37")
+					(reference "R25")
 					(unit 1)
 				)
@@
 		(dnp no)
 		(fields_autoplaced yes)
-		(property "Reference" "R35"
+		(property "Reference" "R23"
 			(at 115.57 71.1199 0)
 			(show_name no)
@@
 			(project "controllerBoard"
 				(path "/93a9a1ca-4ee5-40da-ab67-92836146c003/8b3cd8c5-d66b-460c-b4ee-229e25c1238a"
-					(reference "R35")
+					(reference "R23")
 					(unit 1)
 				)
@@
 		(dnp no)
 		(fields_autoplaced yes)
-		(property "Reference" "#PWR0100"
+		(property "Reference" "#PWR094"
 			(at 88.9 90.17 0)
 			(hide yes)
@@
 			(project "controllerBoard"
 				(path "/93a9a1ca-4ee5-40da-ab67-92836146c003/8b3cd8c5-d66b-460c-b4ee-229e25c1238a"
-					(reference "#PWR0100")
+					(reference "#PWR094")
 					(unit 1)
 				)
@@
 		(dnp no)
 		(fields_autoplaced yes)
-		(property "Reference" "#PWR0108"
+		(property "Reference" "#PWR0102"
 			(at 187.96 100.33 0)
 			(hide yes)
@@
 			(project "controllerBoard"
 				(path "/93a9a1ca-4ee5-40da-ab67-92836146c003/8b3cd8c5-d66b-460c-b4ee-229e25c1238a"
-					(reference "#PWR0108")
+					(reference "#PWR0102")
 					(unit 1)
 				)
@@
 		(dnp no)
 		(fields_autoplaced yes)
-		(property "Reference" "#PWR0104"
+		(property "Reference" "#PWR098"
 			(at 138.43 100.33 0)
 			(hide yes)
@@
 			(project "controllerBoard"
 				(path "/93a9a1ca-4ee5-40da-ab67-92836146c003/8b3cd8c5-d66b-460c-b4ee-229e25c1238a"
-					(reference "#PWR0104")
+					(reference "#PWR098")
 					(unit 1)
 				)
@@
 		(dnp no)
 		(fields_autoplaced yes)
-		(property "Reference" "R38"
+		(property "Reference" "R26"
 			(at 165.1 71.1199 0)
 			(show_name no)
@@
 			(project "controllerBoard"
 				(path "/93a9a1ca-4ee5-40da-ab67-92836146c003/8b3cd8c5-d66b-460c-b4ee-229e25c1238a"
-					(reference "R38")
+					(reference "R26")
 					(unit 1)
 				)
@@
 		(dnp no)
 		(fields_autoplaced yes)
-		(property "Reference" "Q412"
+		(property "Reference" "Q405"
 			(at 116.84 62.2299 0)
 			(show_name no)
@@
 			(project "controllerBoard"
 				(path "/93a9a1ca-4ee5-40da-ab67-92836146c003/8b3cd8c5-d66b-460c-b4ee-229e25c1238a"
-					(reference "Q412")
+					(reference "Q405")
 					(unit 1)
 				)
@@
 		(dnp no)
 		(fields_autoplaced yes)
-		(property "Reference" "R39"
+		(property "Reference" "R27"
 			(at 190.5 71.1199 0)
 			(show_name no)
@@
 			(project "controllerBoard"
 				(path "/93a9a1ca-4ee5-40da-ab67-92836146c003/8b3cd8c5-d66b-460c-b4ee-229e25c1238a"
-					(reference "R39")
+					(reference "R27")
 					(unit 1)
 				)
@@
 		(dnp no)
 		(fields_autoplaced yes)
-		(property "Reference" "#PWR0107"
+		(property "Reference" "#PWR0101"
 			(at 162.56 100.33 0)
 			(hide yes)
@@
 			(project "controllerBoard"
 				(path "/93a9a1ca-4ee5-40da-ab67-92836146c003/8b3cd8c5-d66b-460c-b4ee-229e25c1238a"
-					(reference "#PWR0107")
-					(unit 1)
-				)
+					(reference "#PWR0101")
+					(unit 1)
+				)
