File: kicad/sramBoard/1_16_5V_DEMUX_NOTOUT/5VNOT/5VNOT.kicad_sch (KiCad schematic)
At the start: 2 parts, among them Q1025 PMOS, Q1026 NMOS

Commit message: cdcdcdcdcdcdcdcdcdcdc
Parts:
- Q1025: footprint Package_TO_SOT_SMD:SOT-23 -> easyeda2kicad:SOT-23-P
- Q1026: footprint Package_TO_SOT_SMD:SOT-23 -> easyeda2kicad:SOT-23-N
Changed lines of the file:
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@@
 			)
 		)
-		(property "Footprint" "Package_TO_SOT_SMD:SOT-23"
+		(property "Footprint" "easyeda2kicad:SOT-23-N"
 			(at 119.38 67.31 0)
 			(hide yes)
@@
 			)
 		)
-		(property "Footprint" "Package_TO_SOT_SMD:SOT-23"
+		(property "Footprint" "easyeda2kicad:SOT-23-P"
 			(at 119.38 57.15 0)
 			(hide yes)

Commit message: finish main pcb
Parts:
- Q1153: renamed from Q1025; LCSC Part # (none) -> C41384537
- Q1154: renamed from Q1026; LCSC Part # (none) -> C49308282
Changed lines of the file:
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@@
 		(dnp no)
 		(fields_autoplaced yes)
-		(property "Reference" "Q1026"
+		(property "Reference" "Q1154"
 			(at 120.65 68.5799 0)
 			(show_name no)
@@
 		(property "Sim.Pins" "1=D 2=G 3=S"
 			(at 114.3 85.09 0)
+			(hide yes)
+			(show_name no)
+			(do_not_autoplace no)
+			(effects
+				(font
+					(size 1.27 1.27)
+				)
+			)
+		)
+		(property "LCSC Part #" "C49308282"
+			(at 114.3 69.85 0)
 			(hide yes)
 			(show_name no)
@@
 			(project "sramBoard"
 				(path "/13380198-0e23-4241-a844-cca11526fb8d/a0132d23-2efe-4baa-845a-d59f49944fa0/0600d891-ccd3-4602-9849-fea3d7e045ca"
-					(reference "Q1032")
+					(reference "Q1160")
 					(unit 1)
 				)
 				(path "/13380198-0e23-4241-a844-cca11526fb8d/a0132d23-2efe-4baa-845a-d59f49944fa0/2e151ebf-7913-49eb-83f7-10f1b73fc84d"
-					(reference "Q1030")
+					(reference "Q1158")
 					(unit 1)
 				)
 				(path "/13380198-0e23-4241-a844-cca11526fb8d/a0132d23-2efe-4baa-845a-d59f49944fa0/40364bbe-d9b2-4f0d-a83e-984d8754432c"
-					(reference "Q1026")
+					(reference "Q1154")
 					(unit 1)
 				)
 				(path "/13380198-0e23-4241-a844-cca11526fb8d/a0132d23-2efe-4baa-845a-d59f49944fa0/afd2047a-5605-416e-9801-fddbd3089131"
-					(reference "Q1028")
+					(reference "Q1156")
 					(unit 1)
 				)
@@
 		(dnp no)
 		(fields_autoplaced yes)
-		(property "Reference" "#PWR0260"
+		(property "Reference" "#PWR0516"
 			(at 116.84 53.34 0)
 			(hide yes)
@@
 			(project "sramBoard"
 				(path "/13380198-0e23-4241-a844-cca11526fb8d/a0132d23-2efe-4baa-845a-d59f49944fa0/0600d891-ccd3-4602-9849-fea3d7e045ca"
-					(reference "#PWR0266")
+					(reference "#PWR0522")
 					(unit 1)
 				)
 				(path "/13380198-0e23-4241-a844-cca11526fb8d/a0132d23-2efe-4baa-845a-d59f49944fa0/2e151ebf-7913-49eb-83f7-10f1b73fc84d"
-					(reference "#PWR0264")
+					(reference "#PWR0520")
 					(unit 1)
 				)
 				(path "/13380198-0e23-4241-a844-cca11526fb8d/a0132d23-2efe-4baa-845a-d59f49944fa0/40364bbe-d9b2-4f0d-a83e-984d8754432c"
-					(reference "#PWR0260")
+					(reference "#PWR0516")
 					(unit 1)
 				)
 				(path "/13380198-0e23-4241-a844-cca11526fb8d/a0132d23-2efe-4baa-845a-d59f49944fa0/afd2047a-5605-416e-9801-fddbd3089131"
-					(reference "#PWR0262")
+					(reference "#PWR0518")
 					(unit 1)
 				)
@@
 		(dnp no)
 		(fields_autoplaced yes)
-		(property "Reference" "Q1025"
+		(property "Reference" "Q1153"
 			(at 120.65 53.3399 0)
 			(show_name no)
@@
 		(property "Sim.Pins" "1=D 2=G 3=S"
 			(at 114.3 39.37 0)
+			(hide yes)
+			(show_name no)
+			(do_not_autoplace no)
+			(effects
+				(font
+					(size 1.27 1.27)
+				)
+			)
+		)
+		(property "LCSC Part #" "C41384537"
+			(at 114.3 54.61 0)
 			(hide yes)
 			(show_name no)
@@
 			(project "sramBoard"
 				(path "/13380198-0e23-4241-a844-cca11526fb8d/a0132d23-2efe-4baa-845a-d59f49944fa0/0600d891-ccd3-4602-9849-fea3d7e045ca"
-					(reference "Q1031")
+					(reference "Q1159")
 					(unit 1)
 				)
 				(path "/13380198-0e23-4241-a844-cca11526fb8d/a0132d23-2efe-4baa-845a-d59f49944fa0/2e151ebf-7913-49eb-83f7-10f1b73fc84d"
-					(reference "Q1029")
+					(reference "Q1157")
 					(unit 1)
 				)
 				(path "/13380198-0e23-4241-a844-cca11526fb8d/a0132d23-2efe-4baa-845a-d59f49944fa0/40364bbe-d9b2-4f0d-a83e-984d8754432c"
-					(reference "Q1025")
+					(reference "Q1153")
 					(unit 1)
 				)
 				(path "/13380198-0e23-4241-a844-cca11526fb8d/a0132d23-2efe-4baa-845a-d59f49944fa0/afd2047a-5605-416e-9801-fddbd3089131"
-					(reference "Q1027")
+					(reference "Q1155")
 					(unit 1)
 				)
@@
 		(dnp no)
 		(fields_autoplaced yes)
-		(property "Reference" "#PWR0261"
+		(property "Reference" "#PWR0517"
 			(at 116.84 81.28 0)
 			(hide yes)
@@
 			(project "sramBoard"
 				(path "/13380198-0e23-4241-a844-cca11526fb8d/a0132d23-2efe-4baa-845a-d59f49944fa0/0600d891-ccd3-4602-9849-fea3d7e045ca"
-					(reference "#PWR0267")
+					(reference "#PWR0523")
 					(unit 1)
 				)
 				(path "/13380198-0e23-4241-a844-cca11526fb8d/a0132d23-2efe-4baa-845a-d59f49944fa0/2e151ebf-7913-49eb-83f7-10f1b73fc84d"
-					(reference "#PWR0265")
+					(reference "#PWR0521")
 					(unit 1)
 				)
 				(path "/13380198-0e23-4241-a844-cca11526fb8d/a0132d23-2efe-4baa-845a-d59f49944fa0/40364bbe-d9b2-4f0d-a83e-984d8754432c"
-					(reference "#PWR0261")
+					(reference "#PWR0517")
 					(unit 1)
 				)
 				(path "/13380198-0e23-4241-a844-cca11526fb8d/a0132d23-2efe-4baa-845a-d59f49944fa0/afd2047a-5605-416e-9801-fddbd3089131"
-					(reference "#PWR0263")
-					(unit 1)
-				)
+					(reference "#PWR0519")
+					(unit 1)
+				)

Commit message: fix main ram board
Parts:
- Q1153: value PMOS -> Q_PMOS_GSD; symbol Simulation_SPICE:PMOS -> Transistor_FET:Q_PMOS_GSD
- Q1154: value NMOS -> Q_NMOS_GSD; symbol Simulation_SPICE:NMOS -> Transistor_FET:Q_NMOS_GSD
Connections:
- net +5V: now also Q1153.2 (S); no longer Q1153.3 (S)
- net A: now also Q1153.1 (G), Q1154.1 (G); no longer Q1153.2 (G), Q1154.2 (G)
- net GND: now also Q1154.2 (S); no longer Q1154.3 (S)
- net Y: now also Q1153.3 (D), Q1154.3 (D); no longer Q1153.1 (D), Q1154.1 (D)
Changed lines of the file:
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@@
 	)
 	(symbol
-		(lib_id "Simulation_SPICE:NMOS")
+		(lib_id "Transistor_FET:Q_NMOS_GSD")
 		(at 114.3 69.85 0)
 		(unit 1)
@@
 			)
 		)
-		(property "Value" "NMOS"
+		(property "Value" "Q_NMOS_GSD"
 			(at 120.65 71.1199 0)
 			(show_name no)
@@
 				(path "/64c295c1-a690-461e-ae3b-f66cfdb6e72a/afd2047a-5605-416e-9801-fddbd3089131"
 					(reference "Q8")
+					(unit 1)
+				)
+			)
+			(project "5VNOT"
+				(path "/cabc387a-6207-4601-83a6-292a0d885e49"
+					(reference "Q1160")
 					(unit 1)
 				)
@@
 		(dnp no)
 		(fields_autoplaced yes)
-		(property "Reference" "#PWR0516"
+		(property "Reference" "#PWR0648"
 			(at 116.84 53.34 0)
 			(hide yes)
@@
 			(project "sramBoard"
 				(path "/13380198-0e23-4241-a844-cca11526fb8d/a0132d23-2efe-4baa-845a-d59f49944fa0/0600d891-ccd3-4602-9849-fea3d7e045ca"
-					(reference "#PWR0522")
+					(reference "#PWR0654")
 					(unit 1)
 				)
 				(path "/13380198-0e23-4241-a844-cca11526fb8d/a0132d23-2efe-4baa-845a-d59f49944fa0/2e151ebf-7913-49eb-83f7-10f1b73fc84d"
-					(reference "#PWR0520")
+					(reference "#PWR0652")
 					(unit 1)
 				)
 				(path "/13380198-0e23-4241-a844-cca11526fb8d/a0132d23-2efe-4baa-845a-d59f49944fa0/40364bbe-d9b2-4f0d-a83e-984d8754432c"
-					(reference "#PWR0516")
+					(reference "#PWR0648")
 					(unit 1)
 				)
 				(path "/13380198-0e23-4241-a844-cca11526fb8d/a0132d23-2efe-4baa-845a-d59f49944fa0/afd2047a-5605-416e-9801-fddbd3089131"
-					(reference "#PWR0518")
+					(reference "#PWR0650")
 					(unit 1)
 				)
@@
 				)
 			)
+			(project "5VNOT"
+				(path "/cabc387a-6207-4601-83a6-292a0d885e49"
+					(reference "#PWR0522")
+					(unit 1)
+				)
+			)
 		)
 	)
 	(symbol
-		(lib_id "Simulation_SPICE:PMOS")
+		(lib_id "Transistor_FET:Q_PMOS_GSD")
 		(at 114.3 54.61 0)
 		(mirror x)
@@
 			)
 		)
-		(property "Value" "PMOS"
+		(property "Value" "Q_PMOS_GSD"
 			(at 120.65 55.8799 0)
 			(show_name no)
@@
 				(path "/64c295c1-a690-461e-ae3b-f66cfdb6e72a/afd2047a-5605-416e-9801-fddbd3089131"
 					(reference "Q7")
+					(unit 1)
+				)
+			)
+			(project "5VNOT"
+				(path "/cabc387a-6207-4601-83a6-292a0d885e49"
+					(reference "Q1159")
 					(unit 1)
 				)
@@
 		(dnp no)
 		(fields_autoplaced yes)
-		(property "Reference" "#PWR0517"
+		(property "Reference" "#PWR0649"
 			(at 116.84 81.28 0)
 			(hide yes)
@@
 			(project "sramBoard"
 				(path "/13380198-0e23-4241-a844-cca11526fb8d/a0132d23-2efe-4baa-845a-d59f49944fa0/0600d891-ccd3-4602-9849-fea3d7e045ca"
-					(reference "#PWR0523")
+					(reference "#PWR0655")
 					(unit 1)
 				)
 				(path "/13380198-0e23-4241-a844-cca11526fb8d/a0132d23-2efe-4baa-845a-d59f49944fa0/2e151ebf-7913-49eb-83f7-10f1b73fc84d"
-					(reference "#PWR0521")
+					(reference "#PWR0653")
 					(unit 1)
 				)
 				(path "/13380198-0e23-4241-a844-cca11526fb8d/a0132d23-2efe-4baa-845a-d59f49944fa0/40364bbe-d9b2-4f0d-a83e-984d8754432c"
-					(reference "#PWR0517")
+					(reference "#PWR0649")
 					(unit 1)
 				)
 				(path "/13380198-0e23-4241-a844-cca11526fb8d/a0132d23-2efe-4baa-845a-d59f49944fa0/afd2047a-5605-416e-9801-fddbd3089131"
-					(reference "#PWR0519")
+					(reference "#PWR0651")
 					(unit 1)
 				)
@@
 				)
 			)
+			(project "5VNOT"
+				(path "/cabc387a-6207-4601-83a6-292a0d885e49"
+					(reference "#PWR0523")
+					(unit 1)
+				)
+			)
 		)
 	)
+	(sheet_instances
+		(path "/"
+			(page "1")
+		)
+	)
