File: kicad/sramBoard/1_16_5V_DEMUX_NOTOUT/5V_5NAND/5V_5NAND.kicad_sch (KiCad schematic)
At the start: 10 parts, among them Q1043 PMOS, Q1044 PMOS, Q1045 PMOS, Q1046 PMOS, Q1047 PMOS, Q1048 NMOS, Q1049 NMOS, Q1050 NMOS, Q1051 NMOS, Q1052 NMOS

Commit message: first pcb deign for main boards
Parts:
- renumbered Q1043 to Q1033, Q1044 to Q1034, Q1045 to Q1035, Q1046 to Q1036, Q1047 to Q1037, Q1048 to Q1038, Q1049 to Q1039, Q1050 to Q1040, Q1051 to Q1041, Q1052 to Q1042

Commit message: cdcdcdcdcdcdcdcdcdcdc
Parts:
- Q1033, Q1034, Q1035, Q1036, Q1037: footprint Package_TO_SOT_SMD:SOT-23 -> easyeda2kicad:SOT-23-P
- Q1038, Q1039, Q1040, Q1041, Q1042: footprint Package_TO_SOT_SMD:SOT-23 -> easyeda2kicad:SOT-23-N
Changed lines of the file:
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@@
 			)
 		)
-		(property "Footprint" "Package_TO_SOT_SMD:SOT-23"
+		(property "Footprint" "easyeda2kicad:SOT-23-N"
 			(at 129.54 90.17 0)
 			(hide yes)
@@
 			)
 		)
-		(property "Footprint" "Package_TO_SOT_SMD:SOT-23"
+		(property "Footprint" "easyeda2kicad:SOT-23-N"
 			(at 129.54 100.33 0)
 			(hide yes)
@@
 			)
 		)
-		(property "Footprint" "Package_TO_SOT_SMD:SOT-23"
+		(property "Footprint" "easyeda2kicad:SOT-23-P"
 			(at 49.53 55.88 0)
 			(hide yes)
@@
 			)
 		)
-		(property "Footprint" "Package_TO_SOT_SMD:SOT-23"
+		(property "Footprint" "easyeda2kicad:SOT-23-N"
 			(at 129.54 80.01 0)
 			(hide yes)
@@
 			)
 		)
-		(property "Footprint" "Package_TO_SOT_SMD:SOT-23"
+		(property "Footprint" "easyeda2kicad:SOT-23-N"
 			(at 129.54 69.85 0)
 			(hide yes)
@@
 			)
 		)
-		(property "Footprint" "Package_TO_SOT_SMD:SOT-23"
+		(property "Footprint" "easyeda2kicad:SOT-23-P"
 			(at 129.54 55.88 0)
 			(hide yes)
@@
 			)
 		)
-		(property "Footprint" "Package_TO_SOT_SMD:SOT-23"
+		(property "Footprint" "easyeda2kicad:SOT-23-P"
 			(at 88.9 55.88 0)
 			(hide yes)
@@
 			)
 		)
-		(property "Footprint" "Package_TO_SOT_SMD:SOT-23"
+		(property "Footprint" "easyeda2kicad:SOT-23-P"
 			(at 109.22 55.88 0)
 			(hide yes)
@@
 			)
 		)
-		(property "Footprint" "Package_TO_SOT_SMD:SOT-23"
+		(property "Footprint" "easyeda2kicad:SOT-23-N"
 			(at 129.54 110.49 0)
 			(hide yes)
@@
 			)
 		)
-		(property "Footprint" "Package_TO_SOT_SMD:SOT-23"
+		(property "Footprint" "easyeda2kicad:SOT-23-P"
 			(at 69.85 55.88 0)
 			(hide yes)

Commit message: finish main pcb
Parts:
- Q1161: renamed from Q1033; LCSC Part # (none) -> C41384537
- Q1162: renamed from Q1034; LCSC Part # (none) -> C41384537
- Q1163: renamed from Q1035; LCSC Part # (none) -> C41384537
- Q1164: renamed from Q1036; LCSC Part # (none) -> C41384537
- Q1165: renamed from Q1037; LCSC Part # (none) -> C41384537
- Q1166: renamed from Q1038; LCSC Part # (none) -> C49308282
- Q1167: renamed from Q1039; LCSC Part # (none) -> C49308282
- Q1168: renamed from Q1040; LCSC Part # (none) -> C49308282
- Q1169: renamed from Q1041; LCSC Part # (none) -> C49308282
- Q1170: renamed from Q1042; LCSC Part # (none) -> C49308282

Commit message: fix main ram board
Parts:
- Q1161, Q1162, Q1163, Q1164, Q1165: value PMOS -> Q_PMOS_GSD; symbol Simulation_SPICE:PMOS -> Transistor_FET:Q_PMOS_GSD
- Q1166, Q1167, Q1168, Q1169, Q1170: value NMOS -> Q_NMOS_GSD; symbol Simulation_SPICE:NMOS -> Transistor_FET:Q_NMOS_GSD
Connections:
- net +5V: now also Q1161.2 (S), Q1162.2 (S), Q1163.2 (S), Q1164.2 (S), Q1165.2 (S); no longer Q1161.3 (S), Q1162.3 (S), Q1163.3 (S), Q1164.3 (S), Q1165.3 (S)
- net A_{0}: now also Q1165.1 (G), Q1166.1 (G); no longer Q1165.2 (G), Q1166.2 (G)
- net A_{1}: now also Q1164.1 (G), Q1167.1 (G); no longer Q1164.2 (G), Q1167.2 (G)
- net A_{2}: now also Q1163.1 (G), Q1168.1 (G); no longer Q1163.2 (G), Q1168.2 (G)
- net A_{3}: now also Q1162.1 (G), Q1169.1 (G); no longer Q1162.2 (G), Q1169.2 (G)
- net A_{4}: now also Q1161.1 (G), Q1170.1 (G); no longer Q1161.2 (G), Q1170.2 (G)
- net GND: now also Q1170.2 (S); no longer Q1170.3 (S)
- net Y: now also Q1161.3 (D), Q1162.3 (D), Q1163.3 (D), Q1164.3 (D), Q1165.3 (D), Q1166.3 (D); no longer Q1161.1 (D), Q1162.1 (D), Q1163.1 (D), Q1164.1 (D), Q1165.1 (D), Q1166.1 (D)
- net at Q1167.3 (D): now also Q1166.2 (S); no longer Q1168.1 (D)
- net at Q1168.3 (D): now also Q1167.2 (S); no longer Q1169.1 (D)
- net at Q1169.3 (D): now also Q1168.2 (S); no longer Q1170.1 (D)
- new net: Q1169.2 (S), Q1170.3 (D)
Changed lines of the file:
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@@
 	)
 	(symbol
-		(lib_id "Simulation_SPICE:NMOS")
+		(lib_id "Transistor_FET:Q_NMOS_GSD")
 		(at 124.46 92.71 0)
 		(unit 1)
@@
 			)
 		)
-		(property "Value" "NMOS"
+		(property "Value" "Q_NMOS_GSD"
 			(at 130.81 93.9799 0)
 			(show_name no)
@@
 	)
 	(symbol
-		(lib_id "Simulation_SPICE:NMOS")
+		(lib_id "Transistor_FET:Q_NMOS_GSD")
 		(at 124.46 102.87 0)
 		(unit 1)
@@
 			)
 		)
-		(property "Value" "NMOS"
+		(property "Value" "Q_NMOS_GSD"
 			(at 130.81 104.1399 0)
 			(show_name no)
@@
 	)
 	(symbol
-		(lib_id "Simulation_SPICE:PMOS")
+		(lib_id "Transistor_FET:Q_PMOS_GSD")
 		(at 44.45 53.34 0)
 		(mirror x)
@@
 			)
 		)
-		(property "Value" "PMOS"
+		(property "Value" "Q_PMOS_GSD"
 			(at 50.8 54.6099 0)
 			(show_name no)
@@
 	)
 	(symbol
-		(lib_id "Simulation_SPICE:NMOS")
+		(lib_id "Transistor_FET:Q_NMOS_GSD")
 		(at 124.46 82.55 0)
 		(unit 1)
@@
 			)
 		)
-		(property "Value" "NMOS"
+		(property "Value" "Q_NMOS_GSD"
 			(at 130.81 83.8199 0)
 			(show_name no)
@@
 		(dnp no)
 		(fields_autoplaced yes)
-		(property "Reference" "#PWR0525"
+		(property "Reference" "#PWR0657"
 			(at 127 124.46 0)
 			(hide yes)
@@
 			(project "sramBoard"
 				(path "/13380198-0e23-4241-a844-cca11526fb8d/a0132d23-2efe-4baa-845a-d59f49944fa0/00a5238f-a54e-4948-8b28-7676fff079b4"
-					(reference "#PWR0543")
+					(reference "#PWR0675")
 					(unit 1)
 				)
 				(path "/13380198-0e23-4241-a844-cca11526fb8d/a0132d23-2efe-4baa-845a-d59f49944fa0/0cf35835-4f43-4f49-83f0-8bc61e27d2c6"
-					(reference "#PWR0547")
+					(reference "#PWR0679")
 					(unit 1)
 				)
 				(path "/13380198-0e23-4241-a844-cca11526fb8d/a0132d23-2efe-4baa-845a-d59f49944fa0/1676bd35-adc0-4874-a7f6-b70bbd103e35"
-					(reference "#PWR0533")
+					(reference "#PWR0665")
 					(unit 1)
 				)
 				(path "/13380198-0e23-4241-a844-cca11526fb8d/a0132d23-2efe-4baa-845a-d59f49944fa0/197ed47d-8726-46d7-a907-c292257605d7"
-					(reference "#PWR0541")
+					(reference "#PWR0673")
 					(unit 1)
 				)
 				(path "/13380198-0e23-4241-a844-cca11526fb8d/a0132d23-2efe-4baa-845a-d59f49944fa0/26f0fc5f-c7cc-4917-905b-7d5d20a490c8"
-					(reference "#PWR0527")
+					(reference "#PWR0659")
 					(unit 1)
 				)
 				(path "/13380198-0e23-4241-a844-cca11526fb8d/a0132d23-2efe-4baa-845a-d59f49944fa0/51cefb6d-daac-49d6-93d0-5f1607581d0b"
-					(reference "#PWR0555")
+					(reference "#PWR0687")
 					(unit 1)
 				)
 				(path "/13380198-0e23-4241-a844-cca11526fb8d/a0132d23-2efe-4baa-845a-d59f49944fa0/5670ff8e-a062-4fcb-a569-136066aead2d"
-					(reference "#PWR0535")
+					(reference "#PWR0667")
 					(unit 1)
 				)
 				(path "/13380198-0e23-4241-a844-cca11526fb8d/a0132d23-2efe-4baa-845a-d59f49944fa0/5bcb3992-c452-4a11-8be8-1bad9b347916"
-					(reference "#PWR0537")
+					(reference "#PWR0669")
 					(unit 1)
 				)
 				(path "/13380198-0e23-4241-a844-cca11526fb8d/a0132d23-2efe-4baa-845a-d59f49944fa0/73400315-9a9b-482c-89f2-3dc05eddf230"
-					(reference "#PWR0525")
+					(reference "#PWR0657")
 					(unit 1)
 				)
 				(path "/13380198-0e23-4241-a844-cca11526fb8d/a0132d23-2efe-4baa-845a-d59f49944fa0/8d8bddb8-7e57-4c39-9d5b-e5dc54e8ecce"
-					(reference "#PWR0551")
+					(reference "#PWR0683")
 					(unit 1)
 				)
 				(path "/13380198-0e23-4241-a844-cca11526fb8d/a0132d23-2efe-4baa-845a-d59f49944fa0/af6dac8e-cbf1-40c9-a8b1-d2993a8349c8"
-					(reference "#PWR0545")
+					(reference "#PWR0677")
 					(unit 1)
 				)
 				(path "/13380198-0e23-4241-a844-cca11526fb8d/a0132d23-2efe-4baa-845a-d59f49944fa0/b152f43e-4bcf-468f-9875-026c814ffa29"
-					(reference "#PWR0553")
+					(reference "#PWR0685")
 					(unit 1)
 				)
 				(path "/13380198-0e23-4241-a844-cca11526fb8d/a0132d23-2efe-4baa-845a-d59f49944fa0/bea89456-5e56-4436-8de4-f0968e71580c"
-					(reference "#PWR0539")
+					(reference "#PWR0671")
 					(unit 1)
 				)
 				(path "/13380198-0e23-4241-a844-cca11526fb8d/a0132d23-2efe-4baa-845a-d59f49944fa0/ce2ea598-e429-4d38-aa7d-4e5f8e5963e2"
-					(reference "#PWR0529")
+					(reference "#PWR0661")
 					(unit 1)
 				)
 				(path "/13380198-0e23-4241-a844-cca11526fb8d/a0132d23-2efe-4baa-845a-d59f49944fa0/d916ecc5-9d3c-47bc-9f14-309ae314b1ef"
-					(reference "#PWR0531")
+					(reference "#PWR0663")
 					(unit 1)
 				)
 				(path "/13380198-0e23-4241-a844-cca11526fb8d/a0132d23-2efe-4baa-845a-d59f49944fa0/f9e1110c-5985-48d3-9125-5456e73e29d6"
-					(reference "#PWR0549")
+					(reference "#PWR0681")
 					(unit 1)
 				)
@@
 		(dnp no)
 		(fields_autoplaced yes)
-		(property "Reference" "#PWR0524"
+		(property "Reference" "#PWR0656"
 			(at 127 41.91 0)
 			(hide yes)
@@
 			(project "sramBoard"
 				(path "/13380198-0e23-4241-a844-cca11526fb8d/a0132d23-2efe-4baa-845a-d59f49944fa0/00a5238f-a54e-4948-8b28-7676fff079b4"
-					(reference "#PWR0542")
+					(reference "#PWR0674")
 					(unit 1)
 				)
 				(path "/13380198-0e23-4241-a844-cca11526fb8d/a0132d23-2efe-4baa-845a-d59f49944fa0/0cf35835-4f43-4f49-83f0-8bc61e27d2c6"
-					(reference "#PWR0546")
+					(reference "#PWR0678")
 					(unit 1)
 				)
 				(path "/13380198-0e23-4241-a844-cca11526fb8d/a0132d23-2efe-4baa-845a-d59f49944fa0/1676bd35-adc0-4874-a7f6-b70bbd103e35"
-					(reference "#PWR0532")
+					(reference "#PWR0664")
 					(unit 1)
 				)
 				(path "/13380198-0e23-4241-a844-cca11526fb8d/a0132d23-2efe-4baa-845a-d59f49944fa0/197ed47d-8726-46d7-a907-c292257605d7"
-					(reference "#PWR0540")
+					(reference "#PWR0672")
 					(unit 1)
 				)
 				(path "/13380198-0e23-4241-a844-cca11526fb8d/a0132d23-2efe-4baa-845a-d59f49944fa0/26f0fc5f-c7cc-4917-905b-7d5d20a490c8"
-					(reference "#PWR0526")
+					(reference "#PWR0658")
 					(unit 1)
 				)
 				(path "/13380198-0e23-4241-a844-cca11526fb8d/a0132d23-2efe-4baa-845a-d59f49944fa0/51cefb6d-daac-49d6-93d0-5f1607581d0b"
-					(reference "#PWR0554")
+					(reference "#PWR0686")
 					(unit 1)
 				)
 				(path "/13380198-0e23-4241-a844-cca11526fb8d/a0132d23-2efe-4baa-845a-d59f49944fa0/5670ff8e-a062-4fcb-a569-136066aead2d"
-					(reference "#PWR0534")
+					(reference "#PWR0666")
 					(unit 1)
 				)
 				(path "/13380198-0e23-4241-a844-cca11526fb8d/a0132d23-2efe-4baa-845a-d59f49944fa0/5bcb3992-c452-4a11-8be8-1bad9b347916"
-					(reference "#PWR0536")
+					(reference "#PWR0668")
 					(unit 1)
 				)
 				(path "/13380198-0e23-4241-a844-cca11526fb8d/a0132d23-2efe-4baa-845a-d59f49944fa0/73400315-9a9b-482c-89f2-3dc05eddf230"
-					(reference "#PWR0524")
+					(reference "#PWR0656")
 					(unit 1)
 				)
 				(path "/13380198-0e23-4241-a844-cca11526fb8d/a0132d23-2efe-4baa-845a-d59f49944fa0/8d8bddb8-7e57-4c39-9d5b-e5dc54e8ecce"
-					(reference "#PWR0550")
+					(reference "#PWR0682")
 					(unit 1)
 				)
 				(path "/13380198-0e23-4241-a844-cca11526fb8d/a0132d23-2efe-4baa-845a-d59f49944fa0/af6dac8e-cbf1-40c9-a8b1-d2993a8349c8"
-					(reference "#PWR0544")
+					(reference "#PWR0676")
 					(unit 1)
 				)
 				(path "/13380198-0e23-4241-a844-cca11526fb8d/a0132d23-2efe-4baa-845a-d59f49944fa0/b152f43e-4bcf-468f-9875-026c814ffa29"
-					(reference "#PWR0552")
+					(reference "#PWR0684")
 					(unit 1)
 				)
 				(path "/13380198-0e23-4241-a844-cca11526fb8d/a0132d23-2efe-4baa-845a-d59f49944fa0/bea89456-5e56-4436-8de4-f0968e71580c"
-					(reference "#PWR0538")
+					(reference "#PWR0670")
 					(unit 1)
 				)
 				(path "/13380198-0e23-4241-a844-cca11526fb8d/a0132d23-2efe-4baa-845a-d59f49944fa0/ce2ea598-e429-4d38-aa7d-4e5f8e5963e2"
-					(reference "#PWR0528")
+					(reference "#PWR0660")
 					(unit 1)
 				)
 				(path "/13380198-0e23-4241-a844-cca11526fb8d/a0132d23-2efe-4baa-845a-d59f49944fa0/d916ecc5-9d3c-47bc-9f14-309ae314b1ef"
-					(reference "#PWR0530")
+					(reference "#PWR0662")
 					(unit 1)
 				)
 				(path "/13380198-0e23-4241-a844-cca11526fb8d/a0132d23-2efe-4baa-845a-d59f49944fa0/f9e1110c-5985-48d3-9125-5456e73e29d6"
-					(reference "#PWR0548")
+					(reference "#PWR0680")
 					(unit 1)
 				)
@@
 	)
 	(symbol
-		(lib_id "Simulation_SPICE:NMOS")
+		(lib_id "Transistor_FET:Q_NMOS_GSD")
 		(at 124.46 72.39 0)
 		(unit 1)
@@
 			)
 		)
-		(property "Value" "NMOS"
+		(property "Value" "Q_NMOS_GSD"
 			(at 130.81 73.6599 0)
 			(show_name no)
@@
 	)
 	(symbol
-		(lib_id "Simulation_SPICE:PMOS")
+		(lib_id "Transistor_FET:Q_PMOS_GSD")
 		(at 124.46 53.34 0)
 		(mirror x)
@@
 			)
 		)
-		(property "Value" "PMOS"
+		(property "Value" "Q_PMOS_GSD"
 			(at 130.81 54.6099 0)
 			(show_name no)
@@
 	)
 	(symbol
-		(lib_id "Simulation_SPICE:PMOS")
+		(lib_id "Transistor_FET:Q_PMOS_GSD")
 		(at 83.82 53.34 0)
 		(mirror x)
@@
 			)
 		)
-		(property "Value" "PMOS"
+		(property "Value" "Q_PMOS_GSD"
 			(at 90.17 54.6099 0)
 			(show_name no)
@@
 	)
 	(symbol
-		(lib_id "Simulation_SPICE:PMOS")
+		(lib_id "Transistor_FET:Q_PMOS_GSD")
 		(at 104.14 53.34 0)
 		(mirror x)
@@
 			)
 		)
-		(property "Value" "PMOS"
+		(property "Value" "Q_PMOS_GSD"
 			(at 110.49 54.6099 0)
 			(show_name no)
@@
 	)
 	(symbol
-		(lib_id "Simulation_SPICE:NMOS")
+		(lib_id "Transistor_FET:Q_NMOS_GSD")
 		(at 124.46 113.03 0)
 		(unit 1)
@@
 			)
 		)
-		(property "Value" "NMOS"
+		(property "Value" "Q_NMOS_GSD"
 			(at 130.81 114.2999 0)
 			(show_name no)
@@
 	)
 	(symbol
-		(lib_id "Simulation_SPICE:PMOS")
+		(lib_id "Transistor_FET:Q_PMOS_GSD")
 		(at 64.77 53.34 0)
 		(mirror x)
@@
 			)
 		)
-		(property "Value" "PMOS"
+		(property "Value" "Q_PMOS_GSD"
 			(at 71.12 54.6099 0)
 			(show_name no)
