File: kicad/sramBoard/LOGIC_TO_WL_LEVEL_SHIFT/LOGIC_TO_WL_LEVEL_SHIFT.kicad_sch (KiCad schematic)
At the start: 32 parts, among them Q1193 PMOS, Q1194 NMOS, Q1195 PMOS, Q1196 NMOS, Q1197 PMOS, Q1198 NMOS, Q1199 PMOS, Q1200 NMOS, Q1201 PMOS, Q1202 NMOS, Q1203 PMOS, Q1204 NMOS, Q1205 PMOS, Q1206 NMOS, Q1207 PMOS, Q1208 NMOS, Q1209 PMOS, Q1210 NMOS, Q1211 PMOS, Q1212 NMOS, Q1213 PMOS, Q1214 NMOS, Q1215 PMOS, Q1216 NMOS, Q1217 PMOS, Q1218 NMOS, Q1219 PMOS, Q1220 NMOS, Q1221 PMOS, Q1222 NMOS, Q1223 PMOS, Q1224 NMOS

Commit message: first pcb deign for main boards
Parts:
- renumbered Q1209 to Q1195, Q1210 to Q1196, Q1195 to Q1197, Q1196 to Q1198, Q1211 to Q1199, Q1212 to Q1200, Q1197 to Q1201, Q1198 to Q1202, Q1213 to Q1203, Q1214 to Q1204, Q1199 to Q1205, Q1200 to Q1206, Q1215 to Q1207, Q1216 to Q1208, Q1201 to Q1209, Q1202 to Q1210, Q1217 to Q1211, Q1218 to Q1212, Q1203 to Q1213, Q1204 to Q1214, Q1219 to Q1215, Q1220 to Q1216, Q1205 to Q1217, Q1206 to Q1218, Q1221 to Q1219, Q1222 to Q1220, Q1207 to Q1221, Q1208 to Q1222
Connections:
- net +10V: now reaches Q1193.3 (S), Q1195.3 (S), Q1197.3 (S), Q1199.3 (S), Q1201.3 (S), Q1203.3 (S), Q1205.3 (S), Q1207.3 (S), Q1209.3 (S), Q1211.3 (S), Q1213.3 (S), Q1215.3 (S), Q1217.3 (S), Q1219.3 (S), Q1221.3 (S), Q1223.3 (S)

Commit message: cdcdcdcdcdcdcdcdcdcdc
Parts:
- removed Q1193, Q1195, Q1197, Q1199, Q1201, Q1203, Q1205, Q1207, Q1209, Q1211, Q1213, Q1215, Q1217, Q1219, Q1221, Q1223: PMOS, Package_TO_SOT_SMD:SOT-23, symbol Simulation_SPICE:PMOS
- added R1, R10, R11, R12, R13, R14, R15, R16, R2, R3, R4, R5, R6, R7, R8, R9: 10kR, Resistor_SMD:R_0603_1608Metric, symbol Device:R
- Q1194, Q1196, Q1198, Q1200, Q1202, Q1204, Q1206, Q1208, Q1210, Q1212, Q1214, Q1216, Q1218, Q1220, Q1222, Q1224: footprint Package_TO_SOT_SMD:SOT-23 -> easyeda2kicad:SOT-23-N
Connections:
- net +10V: now also R1.1, R10.1, R11.1, R12.1, R13.1, R14.1, R15.1, R16.1, R2.1, R3.1, R4.1, R5.1, R6.1, R7.1, R8.1, R9.1
- net ~{Y_{0}}: now also R1.2
- net ~{Y_{10}}: now also R11.2
- net ~{Y_{11}}: now also R12.2
- net ~{Y_{12}}: now also R13.2
- net ~{Y_{13}}: now also R14.2
- net ~{Y_{14}}: now also R15.2
- net ~{Y_{15}}: now also R16.2
- net ~{Y_{1}}: now also R2.2
- net ~{Y_{2}}: now also R3.2
- net ~{Y_{3}}: now also R4.2
- net ~{Y_{4}}: now also R5.2
- net ~{Y_{5}}: now also R6.2
- net ~{Y_{6}}: now also R7.2
- net ~{Y_{7}}: now also R8.2
- net ~{Y_{8}}: now also R9.2
- net ~{Y_{9}}: now also R10.2

Commit message: add pmos resistors
Parts:
- renumbered Q1194 to Q1193, Q1196 to Q1194, Q1198 to Q1195, Q1200 to Q1196, Q1202 to Q1197, Q1204 to Q1198, Q1206 to Q1199, Q1208 to Q1200, Q1210 to Q1201, Q1212 to Q1202, Q1214 to Q1203, Q1216 to Q1204, Q1218 to Q1205, Q1220 to Q1206, Q1222 to Q1207, Q1224 to Q1208, R1 to R129, R9 to R130, R2 to R131, R10 to R132, R3 to R133, R11 to R134, R4 to R135, R12 to R136, R5 to R137, R13 to R138, R6 to R139, R14 to R140, R7 to R141, R15 to R142, R8 to R143, R16 to R144

Commit message: finish main pcb
Parts:
- Q1321: renamed from Q1193; LCSC Part # (none) -> C49308282
- Q1322: renamed from Q1194; LCSC Part # (none) -> C49308282
- Q1323: renamed from Q1195; LCSC Part # (none) -> C49308282
- Q1324: renamed from Q1196; LCSC Part # (none) -> C49308282
- Q1325: renamed from Q1197; LCSC Part # (none) -> C49308282
- Q1326: renamed from Q1198; LCSC Part # (none) -> C49308282
- Q1327: renamed from Q1199; LCSC Part # (none) -> C49308282
- Q1328: renamed from Q1200; LCSC Part # (none) -> C49308282
- Q1329: renamed from Q1201; LCSC Part # (none) -> C49308282
- Q1330: renamed from Q1202; LCSC Part # (none) -> C49308282
- Q1331: renamed from Q1203; LCSC Part # (none) -> C49308282
- Q1332: renamed from Q1204; LCSC Part # (none) -> C49308282
- Q1333: renamed from Q1205; LCSC Part # (none) -> C49308282
- Q1334: renamed from Q1206; LCSC Part # (none) -> C49308282
- Q1335: renamed from Q1207; LCSC Part # (none) -> C49308282
- Q1336: renamed from Q1208; LCSC Part # (none) -> C49308282
- R257: renamed from R129; LCSC Part # (none) -> C54920960
- R258: renamed from R130; LCSC Part # (none) -> C54920960
- R259: renamed from R131; LCSC Part # (none) -> C54920960
- R260: renamed from R132; LCSC Part # (none) -> C54920960
- R261: renamed from R133; LCSC Part # (none) -> C54920960
- R262: renamed from R134; LCSC Part # (none) -> C54920960
- R263: renamed from R135; LCSC Part # (none) -> C54920960
- R264: renamed from R136; LCSC Part # (none) -> C54920960
- R265: renamed from R137; LCSC Part # (none) -> C54920960
- R266: renamed from R138; LCSC Part # (none) -> C54920960
- R267: renamed from R139; LCSC Part # (none) -> C54920960
- R268: renamed from R140; LCSC Part # (none) -> C54920960
- R269: renamed from R141; LCSC Part # (none) -> C54920960
- R270: renamed from R142; LCSC Part # (none) -> C54920960
- R271: renamed from R143; LCSC Part # (none) -> C54920960
- R272: renamed from R144; LCSC Part # (none) -> C54920960

Commit message: fix main ram board
Parts:
- added C133, C134, C135, C136: 100nC, Capacitor_SMD:C_0603_1608Metric, symbol Device:C
- Q1321, Q1322, Q1323, Q1324, Q1325, Q1326, Q1327, Q1328, Q1329, Q1330, Q1331, Q1332, Q1333, Q1334, Q1335, Q1336: value NMOS -> Q_NMOS_GSD; symbol Simulation_SPICE:NMOS -> Transistor_FET:Q_NMOS_GSD
Connections:
- net +10V: now also C133.1, C134.1, C135.1, C136.1
- net A_{0}: now also Q1321.1 (G); no longer Q1321.2 (G)
- net A_{10}: now also Q1326.1 (G); no longer Q1326.2 (G)
- net A_{11}: now also Q1328.1 (G); no longer Q1328.2 (G)
- net A_{12}: now also Q1330.1 (G); no longer Q1330.2 (G)
- net A_{13}: now also Q1332.1 (G); no longer Q1332.2 (G)
- net A_{14}: now also Q1334.1 (G); no longer Q1334.2 (G)
- net A_{15}: now also Q1336.1 (G); no longer Q1336.2 (G)
- net A_{1}: now also Q1323.1 (G); no longer Q1323.2 (G)
- net A_{2}: now also Q1325.1 (G); no longer Q1325.2 (G)
- net A_{3}: now also Q1327.1 (G); no longer Q1327.2 (G)
- net A_{4}: now also Q1329.1 (G); no longer Q1329.2 (G)
- net A_{5}: now also Q1331.1 (G); no longer Q1331.2 (G)
- net A_{6}: now also Q1333.1 (G); no longer Q1333.2 (G)
- net A_{7}: now also Q1335.1 (G); no longer Q1335.2 (G)
- net A_{8}: now also Q1322.1 (G); no longer Q1322.2 (G)
- net A_{9}: now also Q1324.1 (G); no longer Q1324.2 (G)
- net GND: now also Q1321.2 (S), Q1322.2 (S), Q1323.2 (S), Q1324.2 (S), Q1325.2 (S), Q1326.2 (S), Q1327.2 (S), Q1328.2 (S), Q1329.2 (S), Q1330.2 (S), Q1331.2 (S), Q1332.2 (S), Q1333.2 (S), Q1334.2 (S), Q1335.2 (S), Q1336.2 (S), C133.2, C134.2, C135.2, C136.2; no longer Q1321.3 (S), Q1322.3 (S), Q1323.3 (S), Q1324.3 (S), Q1325.3 (S), Q1326.3 (S), Q1327.3 (S), Q1328.3 (S), Q1329.3 (S), Q1330.3 (S), Q1331.3 (S), Q1332.3 (S), Q1333.3 (S), Q1334.3 (S), Q1335.3 (S), Q1336.3 (S)
- net ~{Y_{0}}: now also Q1321.3 (D); no longer Q1321.1 (D)
- net ~{Y_{10}}: now also Q1326.3 (D); no longer Q1326.1 (D)
- net ~{Y_{11}}: now also Q1328.3 (D); no longer Q1328.1 (D)
- net ~{Y_{12}}: now also Q1330.3 (D); no longer Q1330.1 (D)
- net ~{Y_{13}}: now also Q1332.3 (D); no longer Q1332.1 (D)
- net ~{Y_{14}}: now also Q1334.3 (D); no longer Q1334.1 (D)
- net ~{Y_{15}}: now also Q1336.3 (D); no longer Q1336.1 (D)
- net ~{Y_{1}}: now also Q1323.3 (D); no longer Q1323.1 (D)
- net ~{Y_{2}}: now also Q1325.3 (D); no longer Q1325.1 (D)
- net ~{Y_{3}}: now also Q1327.3 (D); no longer Q1327.1 (D)
- net ~{Y_{4}}: now also Q1329.3 (D); no longer Q1329.1 (D)
- net ~{Y_{5}}: now also Q1331.3 (D); no longer Q1331.1 (D)
- net ~{Y_{6}}: now also Q1333.3 (D); no longer Q1333.1 (D)
- net ~{Y_{7}}: now also Q1335.3 (D); no longer Q1335.1 (D)
- net ~{Y_{8}}: now also Q1322.3 (D); no longer Q1322.1 (D)
- net ~{Y_{9}}: now also Q1324.3 (D); no longer Q1324.1 (D)

Commit message: Add breakout board through holes on main ram board
Parts:
- renumbered R257 to R263, R258 to R264, R259 to R265, R260 to R266, R261 to R267, R262 to R268, R263 to R269, R264 to R270, R265 to R271, R266 to R272, R267 to R273, R268 to R274, R269 to R275, R270 to R276, R271 to R277, R272 to R278
