File: kicad/inputBoard/1CELL/1CELL.kicad_sch (KiCad schematic)
At the start: 4 parts, among them Q1 Q_NMOS_GSD, Q2 Q_NMOS_GSD, SW1 SW_Push, SW2 SW_Push

Commit message: fix journal format and work on a bit of the input
Parts:
- added J1: Conn_01x02_Pin, Connector_PinHeader_1.00mm:PinHeader_1x02_P1.00mm_Vertical, symbol Connector:Conn_01x02_Pin
- renumbered Q2 to Q1, Q1 to Q2, SW2 to SW1, SW1 to SW2
Connections:
- net BL: no longer names the net of Q1.3 (D)
- net BL: now also J1.2 (Pin_2)
- net ~{BL}: no longer names the net of Q2.3 (D)
- net ~{BL}: now also J1.1 (Pin_1)

Commit message: finish main input board
Parts:
- removed Q1, Q2: Q_NMOS_GSD, Package_TO_SOT_SMD:SOT-23, symbol Transistor_FET:Q_NMOS_GSD
Connections:
- net GND: now also SW1.1, SW2.2
- net at J1.1 (Pin_1): now also SW2.1
- net at J1.2 (Pin_2): now also SW1.2
- removed net +5V: SW1.2, SW2.1
Other:
- moved on the sheet: SW1, SW2
