File: kicad/controllerBoard/READ_PULSE_GEN/READ_PULSE_GEN.kicad_sch (KiCad schematic)
At the start: 20 parts, among them Q417 PMOS, Q418 NMOS, Q419 PMOS, Q420 NMOS, Q421 PMOS, Q422 NMOS, Q423 PMOS, Q424 NMOS, Q427 PMOS, Q428 NMOS

Commit message: did stuff
Parts:
- renumbered C5 to C11, C6 to C12, C7 to C13, D3 to D5, Q417 to Q420, Q418 to Q421, Q419 to Q422, Q420 to Q423, Q421 to Q424, Q422 to Q425, Q423 to Q426, Q424 to Q427, Q427 to Q428, Q428 to Q429, R33 to R40, R34 to R41, R35 to R42, R36 to R43, R37 to R44, R38 to R45

Commit message: did more simulation, added bom
Parts:
- R28: renamed from R40; value R -> 47kR
- renumbered C11 to C7, C12 to C8, C13 to C9, D5 to D3, Q420 to Q413, Q421 to Q414, Q422 to Q415, Q423 to Q416, Q424 to Q417, Q425 to Q418, Q426 to Q419, Q427 to Q420, Q428 to Q421, Q429 to Q422, R41 to R29, R42 to R30, R43 to R31, R44 to R32, R45 to R33

Commit message: update main board schematic
Parts:
- C7, C8, C9: footprint (none) -> Capacitor_SMD:C_0805_2012Metric
- Q413, Q415, Q417, Q419, Q421: value PMOS -> Q_PMOS_GSD; footprint (none) -> easyeda2kicad:SOT-23-P; symbol Simulation_SPICE:PMOS -> Transistor_FET:Q_PMOS_GSD
- Q414, Q416, Q418, Q420, Q422: value NMOS -> Q_NMOS_GSD; footprint (none) -> easyeda2kicad:SOT-23-N; symbol Simulation_SPICE:NMOS -> Transistor_FET:Q_NMOS_GSD
- R28, R29, R30, R31, R32, R33: footprint (none) -> Resistor_SMD:R_0805_2012Metric
Connections:
- net +5V: now also Q413.2 (S), Q415.2 (S), Q417.2 (S), Q419.2 (S), Q421.2 (S); no longer Q413.3 (S), Q415.3 (S), Q417.3 (S), Q419.3 (S), Q421.3 (S)
- net GND: now also Q414.2 (S), Q416.2 (S), Q418.2 (S), Q420.2 (S), Q422.2 (S); no longer Q414.3 (S), Q416.3 (S), Q418.3 (S), Q420.3 (S), Q422.3 (S)
- net R_PULSE: now also Q420.3 (D), Q421.1 (G), Q422.1 (G); no longer Q420.1 (D), Q421.2 (G), Q422.2 (G)
- net ~{R_PULSE}: now also Q421.3 (D), Q422.3 (D); no longer Q421.1 (D), Q422.1 (D)
- net at Q417.1 (G): now also C9.2, Q416.3 (D), Q418.1 (G), R31.2; no longer R32.1
- net at C7.2, D3.1 (K), R28.1: now also Q413.1 (G), Q414.1 (G); no longer Q413.2 (G), Q414.2 (G)
- net at R29.1: now also Q413.3 (D); no longer Q413.1 (D)
- net at Q415.1 (G): now also C8.2, Q416.1 (G), R29.2, R30.1; no longer R31.1
- net at R30.2: now also Q414.3 (D); no longer Q414.1 (D)
- net at Q419.1 (G): now also Q418.3 (D), Q420.1 (G), R32.2; no longer R33.1
- new net: Q417.3 (D), R32.1
- new net: Q415.3 (D), R31.1
- new net: Q419.3 (D), R33.1
Changed lines of the file:
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@@
 	)
 	(symbol
-		(lib_id "Simulation_SPICE:PMOS")
+		(lib_id "Transistor_FET:Q_PMOS_GSD")
 		(at 201.93 63.5 0)
 		(mirror x)
@@
 			)
 		)
-		(property "Value" "PMOS"
+		(property "Value" "Q_PMOS_GSD"
 			(at 208.28 64.7699 0)
 			(show_name no)
@@
 			)
 		)
-		(property "Footprint" ""
+		(property "Footprint" "easyeda2kicad:SOT-23-P"
 			(at 207.01 66.04 0)
 			(hide yes)
@@
 	)
 	(symbol
-		(lib_id "Simulation_SPICE:NMOS")
+		(lib_id "Transistor_FET:Q_NMOS_GSD")
 		(at 224.79 88.9 0)
 		(unit 1)
@@
 			)
 		)
-		(property "Value" "NMOS"
+		(property "Value" "Q_NMOS_GSD"
 			(at 231.14 90.1699 0)
 			(show_name no)
@@
 			)
 		)
-		(property "Footprint" ""
+		(property "Footprint" "easyeda2kicad:SOT-23-N"
 			(at 229.87 86.36 0)
 			(hide yes)
@@
 	)
 	(symbol
-		(lib_id "Simulation_SPICE:PMOS")
+		(lib_id "Transistor_FET:Q_PMOS_GSD")
 		(at 245.11 63.5 0)
 		(mirror x)
@@
 			)
 		)
-		(property "Value" "PMOS"
+		(property "Value" "Q_PMOS_GSD"
 			(at 251.46 64.7699 0)
 			(show_name no)
@@
 			)
 		)
-		(property "Footprint" ""
+		(property "Footprint" "easyeda2kicad:SOT-23-P"
 			(at 250.19 66.04 0)
 			(hide yes)
@@
 				)
 			)
+			(project "READ_PULSE_GEN"
+				(path "/aef69c0b-5431-4a1e-8605-60356112db06"
+					(reference "Q421")
+					(unit 1)
+				)
+			)
 		)
 	)
@@
 			)
 		)
-		(property "Footprint" ""
+		(property "Footprint" "Capacitor_SMD:C_0805_2012Metric"
 			(at 113.03 75.2348 0)
 			(hide yes)
@@
 	)
 	(symbol
-		(lib_id "Simulation_SPICE:PMOS")
+		(lib_id "Transistor_FET:Q_PMOS_GSD")
 		(at 138.43 63.5 0)
 		(mirror x)
@@
 			)
 		)
-		(property "Value" "PMOS"
+		(property "Value" "Q_PMOS_GSD"
 			(at 144.78 64.7699 0)
 			(show_name no)
@@
 			)
 		)
-		(property "Footprint" ""
+		(property "Footprint" "easyeda2kicad:SOT-23-P"
 			(at 143.51 66.04 0)
 			(hide yes)
@@
 			)
 		)
-		(property "Footprint" ""
+		(property "Footprint" "Resistor_SMD:R_0805_2012Metric"
 			(at 202.692 72.39 90)
 			(hide yes)
@@
 	)
 	(symbol
-		(lib_id "Simulation_SPICE:PMOS")
+		(lib_id "Transistor_FET:Q_PMOS_GSD")
 		(at 170.18 63.5 0)
 		(mirror x)
@@
 			)
 		)
-		(property "Value" "PMOS"
+		(property "Value" "Q_PMOS_GSD"
 			(at 176.53 64.7699 0)
 			(show_name no)
@@
 			)
 		)
-		(property "Footprint" ""
+		(property "Footprint" "easyeda2kicad:SOT-23-P"
 			(at 175.26 66.04 0)
 			(hide yes)
@@
 	)
 	(symbol
-		(lib_id "Simulation_SPICE:NMOS")
+		(lib_id "Transistor_FET:Q_NMOS_GSD")
 		(at 170.18 88.9 0)
 		(unit 1)
@@
 			)
 		)
-		(property "Value" "NMOS"
+		(property "Value" "Q_NMOS_GSD"
 			(at 176.53 90.1699 0)
 			(show_name no)
@@
 			)
 		)
-		(property "Footprint" ""
+		(property "Footprint" "easyeda2kicad:SOT-23-N"
 			(at 175.26 86.36 0)
 			(hide yes)
@@
 			)
 		)
-		(property "Footprint" ""
+		(property "Footprint" "Resistor_SMD:R_0805_2012Metric"
 			(at 170.942 72.39 90)
 			(hide yes)
@@
 			)
 		)
-		(property "Footprint" ""
+		(property "Footprint" "Resistor_SMD:R_0805_2012Metric"
 			(at 139.192 80.01 90)
 			(hide yes)
@@
 	)
 	(symbol
-		(lib_id "Simulation_SPICE:NMOS")
+		(lib_id "Transistor_FET:Q_NMOS_GSD")
 		(at 201.93 88.9 0)
 		(unit 1)
@@
 			)
 		)
-		(property "Value" "NMOS"
+		(property "Value" "Q_NMOS_GSD"
 			(at 208.28 90.1699 0)
 			(show_name no)
@@
 			)
 		)
-		(property "Footprint" ""
+		(property "Footprint" "easyeda2kicad:SOT-23-N"
 			(at 207.01 86.36 0)
 			(hide yes)
@@
 			)
 		)
-		(property "Footprint" ""
+		(property "Footprint" "Capacitor_SMD:C_0805_2012Metric"
 			(at 181.9148 76.2 0)
 			(hide yes)
@@
 	)
 	(symbol
-		(lib_id "Simulation_SPICE:NMOS")
+		(lib_id "Transistor_FET:Q_NMOS_GSD")
 		(at 245.11 88.9 0)
 		(unit 1)
@@
 			)
 		)
-		(property "Value" "NMOS"
+		(property "Value" "Q_NMOS_GSD"
 			(at 251.46 90.1699 0)
 			(show_name no)
@@
 			)
 		)
-		(property "Footprint" ""
+		(property "Footprint" "easyeda2kicad:SOT-23-N"
 			(at 250.19 86.36 0)
 			(hide yes)
@@
 				)
 			)
+			(project "READ_PULSE_GEN"
+				(path "/aef69c0b-5431-4a1e-8605-60356112db06"
+					(reference "Q422")
+					(unit 1)
+				)
+			)
 		)
 	)
@@
 			)
 		)
-		(property "Footprint" ""
+		(property "Footprint" "Resistor_SMD:R_0805_2012Metric"
 			(at 225.552 72.39 90)
 			(hide yes)
@@
 			)
 		)
-		(property "Footprint" ""
+		(property "Footprint" "Resistor_SMD:R_0805_2012Metric"
 			(at 139.192 72.39 90)
 			(hide yes)
@@
 	)
 	(symbol
-		(lib_id "Simulation_SPICE:NMOS")
+		(lib_id "Transistor_FET:Q_NMOS_GSD")
 		(at 138.43 88.9 0)
 		(unit 1)
@@
 			)
 		)
-		(property "Value" "NMOS"
+		(property "Value" "Q_NMOS_GSD"
 			(at 144.78 90.1699 0)
 			(show_name no)
@@
 			)
 		)
-		(property "Footprint" ""
+		(property "Footprint" "easyeda2kicad:SOT-23-N"
 			(at 143.51 86.36 0)
 			(hide yes)
@@
 				)
 			)
+			(project "READ_PULSE_GEN"
+				(path "/aef69c0b-5431-4a1e-8605-60356112db06"
+					(reference "#PWR0115")
+					(unit 1)
+				)
+			)
 		)
 	)
@@
 				)
 			)
+			(project "READ_PULSE_GEN"
+				(path "/aef69c0b-5431-4a1e-8605-60356112db06"
+					(reference "#PWR0116")
+					(unit 1)
+				)
+			)
 		)
 	)
@@
 			)
 		)
-		(property "Footprint" ""
+		(property "Footprint" "Capacitor_SMD:C_0805_2012Metric"
 			(at 151.4348 76.2 0)
 			(hide yes)
@@
 			)
 		)
-		(property "Footprint" ""
+		(property "Footprint" "Resistor_SMD:R_0805_2012Metric"
 			(at 111.252 80.01 90)
 			(hide yes)
@@
 	)
 	(symbol
-		(lib_id "Simulation_SPICE:PMOS")
+		(lib_id "Transistor_FET:Q_PMOS_GSD")
 		(at 224.79 63.5 0)
 		(mirror x)
@@
 			)
 		)
-		(property "Value" "PMOS"
+		(property "Value" "Q_PMOS_GSD"
 			(at 231.14 64.7699 0)
 			(show_name no)
@@
 			)
 		)
-		(property "Footprint" ""
+		(property "Footprint" "easyeda2kicad:SOT-23-P"
 			(at 229.87 66.04 0)
 			(hide yes)
@@
 		)
 	)
+	(sheet_instances
+		(path "/"
+			(page "1")
+		)
+	)

Commit message: finished routing all sub schematics
Parts:
- renumbered C7 to C11, C8 to C12, C9 to C13
Changed lines of the file:
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@@
 		(dnp no)
 		(fields_autoplaced yes)
-		(property "Reference" "#PWR0109"
+		(property "Reference" "#PWR0111"
 			(at 172.72 100.33 0)
 			(hide yes)
@@
 			(project "controllerBoard"
 				(path "/93a9a1ca-4ee5-40da-ab67-92836146c003/bd8eda89-0d1e-4854-ab6f-a575635da338"
-					(reference "#PWR0109")
+					(reference "#PWR0111")
 					(unit 1)
 				)
@@
 		(dnp no)
 		(fields_autoplaced yes)
-		(property "Reference" "#PWR0114"
+		(property "Reference" "#PWR0116"
 			(at 227.33 100.33 0)
 			(hide yes)
@@
 			(project "controllerBoard"
 				(path "/93a9a1ca-4ee5-40da-ab67-92836146c003/bd8eda89-0d1e-4854-ab6f-a575635da338"
-					(reference "#PWR0114")
+					(reference "#PWR0116")
 					(unit 1)
 				)
@@
 		(dnp no)
 		(fields_autoplaced yes)
-		(property "Reference" "#PWR0106"
+		(property "Reference" "#PWR0108"
 			(at 140.97 100.33 0)
 			(hide yes)
@@
 			(project "controllerBoard"
 				(path "/93a9a1ca-4ee5-40da-ab67-92836146c003/bd8eda89-0d1e-4854-ab6f-a575635da338"
-					(reference "#PWR0106")
+					(reference "#PWR0108")
 					(unit 1)
 				)
@@
 		(dnp no)
 		(fields_autoplaced yes)
-		(property "Reference" "C7"
+		(property "Reference" "C11"
 			(at 109.22 68.58 90)
 			(show_name no)
@@
 			(project "controllerBoard"
 				(path "/93a9a1ca-4ee5-40da-ab67-92836146c003/bd8eda89-0d1e-4854-ab6f-a575635da338"
-					(reference "C7")
+					(reference "C11")
 					(unit 1)
 				)
@@
 		(dnp no)
 		(fields_autoplaced yes)
-		(property "Reference" "#PWR0104"
+		(property "Reference" "#PWR0106"
 			(at 123.19 90.17 0)
 			(hide yes)
@@
 			(project "controllerBoard"
 				(path "/93a9a1ca-4ee5-40da-ab67-92836146c003/bd8eda89-0d1e-4854-ab6f-a575635da338"
-					(reference "#PWR0104")
+					(reference "#PWR0106")
 					(unit 1)
 				)
@@
 		(dnp no)
 		(fields_autoplaced yes)
-		(property "Reference" "#PWR0112"
+		(property "Reference" "#PWR0114"
 			(at 204.47 100.33 0)
 			(hide yes)
@@
 			(project "controllerBoard"
 				(path "/93a9a1ca-4ee5-40da-ab67-92836146c003/bd8eda89-0d1e-4854-ab6f-a575635da338"
-					(reference "#PWR0112")
+					(reference "#PWR0114")
 					(unit 1)
 				)
@@
 		(dnp no)
 		(fields_autoplaced yes)
-		(property "Reference" "#PWR0107"
+		(property "Reference" "#PWR0109"
 			(at 152.4 90.17 0)
 			(hide yes)
@@
 			(project "controllerBoard"
 				(path "/93a9a1ca-4ee5-40da-ab67-92836146c003/bd8eda89-0d1e-4854-ab6f-a575635da338"
-					(reference "#PWR0107")
+					(reference "#PWR0109")
 					(unit 1)
 				)
@@
 		(dnp no)
 		(fields_autoplaced yes)
-		(property "Reference" "#PWR0103"
+		(property "Reference" "#PWR0105"
 			(at 113.03 90.17 0)
 			(hide yes)
@@
 			(project "controllerBoard"
 				(path "/93a9a1ca-4ee5-40da-ab67-92836146c003/bd8eda89-0d1e-4854-ab6f-a575635da338"
-					(reference "#PWR0103")
+					(reference "#PWR0105")
 					(unit 1)
 				)
@@
 		(dnp no)
 		(fields_autoplaced yes)
-		(property "Reference" "#PWR0111"
+		(property "Reference" "#PWR0113"
 			(at 204.47 62.23 0)
 			(hide yes)
@@
 			(project "controllerBoard"
 				(path "/93a9a1ca-4ee5-40da-ab67-92836146c003/bd8eda89-0d1e-4854-ab6f-a575635da338"
-					(reference "#PWR0111")
+					(reference "#PWR0113")
 					(unit 1)
 				)
@@
 		(dnp no)
 		(fields_autoplaced yes)
-		(property "Reference" "#PWR0113"
+		(property "Reference" "#PWR0115"
 			(at 227.33 62.23 0)
 			(hide yes)
@@
 			(project "controllerBoard"
 				(path "/93a9a1ca-4ee5-40da-ab67-92836146c003/bd8eda89-0d1e-4854-ab6f-a575635da338"
-					(reference "#PWR0113")
+					(reference "#PWR0115")
 					(unit 1)
 				)
@@
 		(dnp no)
 		(fields_autoplaced yes)
-		(property "Reference" "C9"
+		(property "Reference" "C13"
 			(at 186.69 78.7399 0)
 			(show_name no)
@@
 			(project "controllerBoard"
 				(path "/93a9a1ca-4ee5-40da-ab67-92836146c003/bd8eda89-0d1e-4854-ab6f-a575635da338"
-					(reference "C9")
+					(reference "C13")
 					(unit 1)
 				)
@@
 		(dnp no)
 		(fields_autoplaced yes)
-		(property "Reference" "#PWR0105"
+		(property "Reference" "#PWR0107"
 			(at 140.97 62.23 0)
 			(hide yes)
@@
 			(project "controllerBoard"
 				(path "/93a9a1ca-4ee5-40da-ab67-92836146c003/bd8eda89-0d1e-4854-ab6f-a575635da338"
-					(reference "#PWR0105")
+					(reference "#PWR0107")
 					(unit 1)
 				)
@@
 		(dnp no)
 		(fields_autoplaced yes)
-		(property "Reference" "#PWR0110"
+		(property "Reference" "#PWR0112"
 			(at 182.88 90.17 0)
 			(hide yes)
@@
 			(project "controllerBoard"
 				(path "/93a9a1ca-4ee5-40da-ab67-92836146c003/bd8eda89-0d1e-4854-ab6f-a575635da338"
-					(reference "#PWR0110")
+					(reference "#PWR0112")
 					(unit 1)
 				)
@@
 		(dnp no)
 		(fields_autoplaced yes)
-		(property "Reference" "#PWR0115"
+		(property "Reference" "#PWR0117"
 			(at 247.65 62.23 0)
 			(hide yes)
@@
 			(project "controllerBoard"
 				(path "/93a9a1ca-4ee5-40da-ab67-92836146c003/bd8eda89-0d1e-4854-ab6f-a575635da338"
-					(reference "#PWR0115")
+					(reference "#PWR0117")
 					(unit 1)
 				)
@@
 		(dnp no)
 		(fields_autoplaced yes)
-		(property "Reference" "#PWR0116"
+		(property "Reference" "#PWR0118"
 			(at 247.65 100.33 0)
 			(hide yes)
@@
 			(project "controllerBoard"
 				(path "/93a9a1ca-4ee5-40da-ab67-92836146c003/bd8eda89-0d1e-4854-ab6f-a575635da338"
-					(reference "#PWR0116")
+					(reference "#PWR0118")
 					(unit 1)
 				)
@@
 		(dnp no)
 		(fields_autoplaced yes)
-		(property "Reference" "#PWR0108"
+		(property "Reference" "#PWR0110"
 			(at 172.72 62.23 0)
 			(hide yes)
@@
 			(project "controllerBoard"
 				(path "/93a9a1ca-4ee5-40da-ab67-92836146c003/bd8eda89-0d1e-4854-ab6f-a575635da338"
-					(reference "#PWR0108")
+					(reference "#PWR0110")
 					(unit 1)
 				)
@@
 		(dnp no)
 		(fields_autoplaced yes)
-		(property "Reference" "C8"
+		(property "Reference" "C12"
 			(at 156.21 78.7399 0)
 			(show_name no)
@@
 			(project "controllerBoard"
 				(path "/93a9a1ca-4ee5-40da-ab67-92836146c003/bd8eda89-0d1e-4854-ab6f-a575635da338"
-					(reference "C8")
-					(unit 1)
-				)
+					(reference "C12")
+					(unit 1)
+				)

Commit message: add mounting holes
Parts:
- renumbered C12 to C10, C13 to C11, C11 to C9
Changed lines of the file:
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@@
 		(dnp no)
 		(fields_autoplaced yes)
-		(property "Reference" "#PWR0111"
+		(property "Reference" "#PWR0161"
 			(at 172.72 100.33 0)
 			(hide yes)
@@
 			(project "controllerBoard"
 				(path "/93a9a1ca-4ee5-40da-ab67-92836146c003/bd8eda89-0d1e-4854-ab6f-a575635da338"
-					(reference "#PWR0111")
+					(reference "#PWR0161")
 					(unit 1)
 				)
@@
 		(dnp no)
 		(fields_autoplaced yes)
-		(property "Reference" "#PWR0116"
+		(property "Reference" "#PWR0166"
 			(at 227.33 100.33 0)
 			(hide yes)
@@
 			(project "controllerBoard"
 				(path "/93a9a1ca-4ee5-40da-ab67-92836146c003/bd8eda89-0d1e-4854-ab6f-a575635da338"
-					(reference "#PWR0116")
+					(reference "#PWR0166")
 					(unit 1)
 				)
@@
 		(dnp no)
 		(fields_autoplaced yes)
-		(property "Reference" "#PWR0108"
+		(property "Reference" "#PWR0158"
 			(at 140.97 100.33 0)
 			(hide yes)
@@
 			(project "controllerBoard"
 				(path "/93a9a1ca-4ee5-40da-ab67-92836146c003/bd8eda89-0d1e-4854-ab6f-a575635da338"
-					(reference "#PWR0108")
+					(reference "#PWR0158")
 					(unit 1)
 				)
@@
 		(dnp no)
 		(fields_autoplaced yes)
-		(property "Reference" "C11"
+		(property "Reference" "C9"
 			(at 109.22 68.58 90)
 			(show_name no)
@@
 			(project "controllerBoard"
 				(path "/93a9a1ca-4ee5-40da-ab67-92836146c003/bd8eda89-0d1e-4854-ab6f-a575635da338"
-					(reference "C11")
+					(reference "C9")
 					(unit 1)
 				)
@@
 		(dnp no)
 		(fields_autoplaced yes)
-		(property "Reference" "#PWR0106"
+		(property "Reference" "#PWR0156"
 			(at 123.19 90.17 0)
 			(hide yes)
@@
 			(project "controllerBoard"
 				(path "/93a9a1ca-4ee5-40da-ab67-92836146c003/bd8eda89-0d1e-4854-ab6f-a575635da338"
-					(reference "#PWR0106")
+					(reference "#PWR0156")
 					(unit 1)
 				)
@@
 		(dnp no)
 		(fields_autoplaced yes)
-		(property "Reference" "#PWR0114"
+		(property "Reference" "#PWR0164"
 			(at 204.47 100.33 0)
 			(hide yes)
@@
 			(project "controllerBoard"
 				(path "/93a9a1ca-4ee5-40da-ab67-92836146c003/bd8eda89-0d1e-4854-ab6f-a575635da338"
-					(reference "#PWR0114")
+					(reference "#PWR0164")
 					(unit 1)
 				)
@@
 		(dnp no)
 		(fields_autoplaced yes)
-		(property "Reference" "#PWR0109"
+		(property "Reference" "#PWR0159"
 			(at 152.4 90.17 0)
 			(hide yes)
@@
 			(project "controllerBoard"
 				(path "/93a9a1ca-4ee5-40da-ab67-92836146c003/bd8eda89-0d1e-4854-ab6f-a575635da338"
-					(reference "#PWR0109")
+					(reference "#PWR0159")
 					(unit 1)
 				)
@@
 		(dnp no)
 		(fields_autoplaced yes)
-		(property "Reference" "#PWR0105"
+		(property "Reference" "#PWR0155"
 			(at 113.03 90.17 0)
 			(hide yes)
@@
 			(project "controllerBoard"
 				(path "/93a9a1ca-4ee5-40da-ab67-92836146c003/bd8eda89-0d1e-4854-ab6f-a575635da338"
-					(reference "#PWR0105")
+					(reference "#PWR0155")
 					(unit 1)
 				)
@@
 		(dnp no)
 		(fields_autoplaced yes)
-		(property "Reference" "#PWR0113"
+		(property "Reference" "#PWR0163"
 			(at 204.47 62.23 0)
 			(hide yes)
@@
 			(project "controllerBoard"
 				(path "/93a9a1ca-4ee5-40da-ab67-92836146c003/bd8eda89-0d1e-4854-ab6f-a575635da338"
-					(reference "#PWR0113")
+					(reference "#PWR0163")
 					(unit 1)
 				)
@@
 		(dnp no)
 		(fields_autoplaced yes)
-		(property "Reference" "#PWR0115"
+		(property "Reference" "#PWR0165"
 			(at 227.33 62.23 0)
 			(hide yes)
@@
 			(project "controllerBoard"
 				(path "/93a9a1ca-4ee5-40da-ab67-92836146c003/bd8eda89-0d1e-4854-ab6f-a575635da338"
-					(reference "#PWR0115")
+					(reference "#PWR0165")
 					(unit 1)
 				)
@@
 		(dnp no)
 		(fields_autoplaced yes)
-		(property "Reference" "C13"
+		(property "Reference" "C11"
 			(at 186.69 78.7399 0)
 			(show_name no)
@@
 			(project "controllerBoard"
 				(path "/93a9a1ca-4ee5-40da-ab67-92836146c003/bd8eda89-0d1e-4854-ab6f-a575635da338"
-					(reference "C13")
+					(reference "C11")
 					(unit 1)
 				)
@@
 		(dnp no)
 		(fields_autoplaced yes)
-		(property "Reference" "#PWR0107"
+		(property "Reference" "#PWR0157"
 			(at 140.97 62.23 0)
 			(hide yes)
@@
 			(project "controllerBoard"
 				(path "/93a9a1ca-4ee5-40da-ab67-92836146c003/bd8eda89-0d1e-4854-ab6f-a575635da338"
-					(reference "#PWR0107")
+					(reference "#PWR0157")
 					(unit 1)
 				)
@@
 		(dnp no)
 		(fields_autoplaced yes)
-		(property "Reference" "#PWR0112"
+		(property "Reference" "#PWR0162"
 			(at 182.88 90.17 0)
 			(hide yes)
@@
 			(project "controllerBoard"
 				(path "/93a9a1ca-4ee5-40da-ab67-92836146c003/bd8eda89-0d1e-4854-ab6f-a575635da338"
-					(reference "#PWR0112")
+					(reference "#PWR0162")
 					(unit 1)
 				)
@@
 		(dnp no)
 		(fields_autoplaced yes)
-		(property "Reference" "#PWR0117"
+		(property "Reference" "#PWR0167"
 			(at 247.65 62.23 0)
 			(hide yes)
@@
 			(project "controllerBoard"
 				(path "/93a9a1ca-4ee5-40da-ab67-92836146c003/bd8eda89-0d1e-4854-ab6f-a575635da338"
-					(reference "#PWR0117")
+					(reference "#PWR0167")
 					(unit 1)
 				)
@@
 		(dnp no)
 		(fields_autoplaced yes)
-		(property "Reference" "#PWR0118"
+		(property "Reference" "#PWR0168"
 			(at 247.65 100.33 0)
 			(hide yes)
@@
 			(project "controllerBoard"
 				(path "/93a9a1ca-4ee5-40da-ab67-92836146c003/bd8eda89-0d1e-4854-ab6f-a575635da338"
-					(reference "#PWR0118")
+					(reference "#PWR0168")
 					(unit 1)
 				)
@@
 		(dnp no)
 		(fields_autoplaced yes)
-		(property "Reference" "#PWR0110"
+		(property "Reference" "#PWR0160"
 			(at 172.72 62.23 0)
 			(hide yes)
@@
 			(project "controllerBoard"
 				(path "/93a9a1ca-4ee5-40da-ab67-92836146c003/bd8eda89-0d1e-4854-ab6f-a575635da338"
-					(reference "#PWR0110")
+					(reference "#PWR0160")
 					(unit 1)
 				)
@@
 		(dnp no)
 		(fields_autoplaced yes)
-		(property "Reference" "C12"
+		(property "Reference" "C10"
 			(at 156.21 78.7399 0)
 			(show_name no)
@@
 			(project "controllerBoard"
 				(path "/93a9a1ca-4ee5-40da-ab67-92836146c003/bd8eda89-0d1e-4854-ab6f-a575635da338"
-					(reference "C12")
-					(unit 1)
-				)
+					(reference "C10")
+					(unit 1)
+				)
