File: kicad/inputBoard/inputBoard.kicad_pcb (KiCad board)
At the start: 2 copper layers, 40 parts, among them J1 Conn_01x02_Pin, J2 Conn_01x02_Pin, J3 Conn_01x02_Pin, J4 Conn_01x02_Pin, J5 Conn_01x02_Pin, J6 Conn_01x02_Pin, J7 Conn_01x02_Pin, J8 Conn_01x02_Pin, Q1 Q_NMOS_GSD, Q10 Q_NMOS_GSD, Q11 Q_NMOS_GSD, Q12 Q_NMOS_GSD, Q13 Q_NMOS_GSD, Q14 Q_NMOS_GSD, Q15 Q_NMOS_GSD, Q16 Q_NMOS_GSD, Q2 Q_NMOS_GSD, Q3 Q_NMOS_GSD, Q4 Q_NMOS_GSD, Q5 Q_NMOS_GSD, Q6 Q_NMOS_GSD, Q7 Q_NMOS_GSD, Q8 Q_NMOS_GSD, Q9 Q_NMOS_GSD, SW1 SW_Push, SW10 SW_Push, SW11 SW_Push, SW12 SW_Push, SW13 SW_Push, SW14 SW_Push, SW15 SW_Push, SW16 SW_Push, SW2 SW_Push, SW3 SW_Push, SW4 SW_Push, SW5 SW_Push, SW6 SW_Push, SW7 SW_Push, SW8 SW_Push, SW9 SW_Push

Commit message: finish main input board
Parts:
- removed Q1, Q10, Q11, Q12, Q13, Q14, Q15, Q16, Q2, Q3, Q4, Q5, Q6, Q7, Q8, Q9: Q_NMOS_GSD, Package_TO_SOT_SMD:SOT-23
- added H1: MountingHole_Pad, MountingHole:MountingHole_2.2mm_M2_DIN965_Pad, F.Cu at (138.4, 81.2)
- added H2: MountingHole_Pad, MountingHole:MountingHole_2.2mm_M2_DIN965_Pad, F.Cu at (164.2, 81.2)
- added H3: MountingHole_Pad, MountingHole:MountingHole_2.2mm_M2_DIN965_Pad, F.Cu at (190.2, 81.3)
- added H4: MountingHole_Pad, MountingHole:MountingHole_2.2mm_M2_DIN965_Pad, F.Cu at (216.1, 81.2)
- added H5: MountingHole_Pad, MountingHole:MountingHole_2.2mm_M2_DIN965_Pad, F.Cu at (241.9, 81.2)
- added R1: 0R, Resistor_SMD:R_1206_3216Metric_Pad1.30x1.75mm_HandSolder, B.Cu at (138.3, 76.2)
- added R2: 0R, Resistor_SMD:R_1206_3216Metric_Pad1.30x1.75mm_HandSolder, B.Cu at (159.4, 80.7)
- added R3: 0R, Resistor_SMD:R_1206_3216Metric_Pad1.30x1.75mm_HandSolder, B.Cu at (185.5, 80.3)
- added R4: 0R, Resistor_SMD:R_1206_3216Metric_Pad1.30x1.75mm_HandSolder, B.Cu at (211.3, 80.0)
- added R5: 0R, Resistor_SMD:R_1206_3216Metric_Pad1.30x1.75mm_HandSolder, B.Cu at (237.2, 80.0)
- moved SW13 173.1 mm to (222.5, 75.4)
- moved J7 172.7 mm to (229.8, 74.1)
- moved SW14 172.5 mm to (222.5, 80.8)
- moved SW16 170.4 mm to (235.4, 80.8)
- moved J8 170.0 mm to (242.7, 74.1)
- moved SW15 169.8 mm to (235.5, 75.4)
- moved SW12 163.6 mm to (209.6, 80.8)
- moved J6 162.5 mm to (216.9, 74.1)
- moved SW11 161.6 mm to (209.6, 75.4)
- moved SW10 120.7 mm to (196.7, 80.8)
- moved J5 119.3 mm to (203.9, 74.1)
- moved SW7 118.9 mm to (183.8, 75.4)
- moved J4 118.3 mm to (191.0, 74.1)
- moved SW8 118.0 mm to (183.8, 80.8)
- moved SW9 118.0 mm to (196.7, 75.4)
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Connections:
- SW1 pad 1: Net-(Q1-G) -> GND
- SW1 pad 2: +5V -> Net-(J1-Pin_2)
- SW10 pad 1: +5V -> Net-(J5-Pin_1)
- SW10 pad 2: Net-(Q10-G) -> GND
- SW11 pad 1: Net-(Q11-G) -> GND
- SW11 pad 2: +5V -> Net-(J6-Pin_2)
- SW12 pad 1: +5V -> Net-(J6-Pin_1)
- SW12 pad 2: Net-(Q12-G) -> GND
- SW13 pad 1: Net-(Q13-G) -> GND
- SW13 pad 2: +5V -> Net-(J7-Pin_2)
- SW14 pad 1: +5V -> Net-(J7-Pin_1)
- SW14 pad 2: Net-(Q14-G) -> GND
- SW15 pad 1: Net-(Q15-G) -> GND
- SW15 pad 2: +5V -> Net-(J8-Pin_2)
- SW16 pad 1: +5V -> Net-(J8-Pin_1)
- SW16 pad 2: Net-(Q16-G) -> GND
- SW2 pad 1: +5V -> Net-(J1-Pin_1)
- SW2 pad 2: Net-(Q2-G) -> GND
- SW3 pad 1: Net-(Q3-G) -> GND
- SW3 pad 2: +5V -> Net-(J2-Pin_2)
- SW4 pad 1: +5V -> Net-(J2-Pin_1)
- SW4 pad 2: Net-(Q4-G) -> GND
- SW5 pad 1: Net-(Q5-G) -> GND
- SW5 pad 2: +5V -> Net-(J3-Pin_2)
- SW6 pad 1: +5V -> Net-(J3-Pin_1)
- SW6 pad 2: Net-(Q6-G) -> GND
- SW7 pad 1: Net-(Q7-G) -> GND
- SW7 pad 2: +5V -> Net-(J4-Pin_2)
- SW8 pad 1: +5V -> Net-(J4-Pin_1)
- SW8 pad 2: Net-(Q8-G) -> GND
- SW9 pad 1: Net-(Q9-G) -> GND
- SW9 pad 2: +5V -> Net-(J5-Pin_2)
Routing:
- net +5V: track 284.2 -> 0.00 mm, vias 8 -> 0
- net GND: track 168.0 -> 72.0 mm
- net Net-(Q14-G): track 12.5 -> 0.00 mm
- net Net-(Q12-G): track 12.5 -> 0.00 mm
- net Net-(Q8-G): track 12.5 -> 0.00 mm
- net Net-(Q4-G): track 12.5 -> 0.00 mm
- net Net-(Q16-G): track 12.5 -> 0.00 mm
- net Net-(Q10-G): track 12.5 -> 0.00 mm
- net Net-(Q2-G): track 12.5 -> 0.00 mm
- net Net-(Q6-G): track 12.5 -> 0.00 mm
- net Net-(J8-Pin_1): track 3.32 -> 12.6 mm
- net Net-(J4-Pin_1): track 3.32 -> 12.6 mm
- net Net-(J7-Pin_1): track 3.32 -> 12.6 mm
- net Net-(J6-Pin_1): track 3.32 -> 12.6 mm
- net Net-(J1-Pin_1): track 3.32 -> 12.6 mm
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- added copper zone on B.Cu, net GND
Other:
- board outline added: 108.3 x 11.3 mm

Commit message: update bom, add more capacitors
Parts:
- added J9: Conn_01x01_Pin, Connector_Wire:Wire_Pad_18AWG_stranded, F.Cu at (228.9, 81.6)
